File: Wsprry-Pi-Synth-Univ/Wsprry-Pi-Synth-Univ.kicad_sch (KiCad schematic)
At the start: 36 parts, among them J11 GPIO, J81 Conn_01x04, J82 Conn_01x04, J83 SMA, SW11 Switch, U51 GVA-84, Y21 ATX-11-F-27.000MHZ-F05-T, Y31 MS5351M

Commit message: Cleanup due to lost libraries
Parts:
- C12, C23, C31, C51: footprint Capacitor_SMD:C_0603_1608Metric -> Wsprry Pi:C_0603_1608Metric; symbol Device:C -> Wsprry Pi:C
- C21, C22, C24, C32, C33, C34, C52, C53: footprint Capacitor_SMD:C_0402_1005Metric -> Wsprry Pi:C_0402_1005Metric; symbol Device:C -> Wsprry Pi:C
- C54, C55: footprint Capacitor_SMD:C_0805_2012Metric -> Wsprry Pi:C_0805_2012Metric; symbol Device:C -> Wsprry Pi:C
- D11: footprint LED_SMD:LED_0603_1608Metric -> Wsprry Pi:LED_0603_1608Metric; symbol Device:LED -> Wsprry Pi:LED
- FB11, FB21, FB31, FB51: footprint Inductor_SMD:L_0603_1608Metric -> Wsprry Pi:L_0603_1608Metric; symbol Device:FerriteBead -> Wsprry Pi:FerriteBead
- J11: footprint Connector_PinSocket_2.54mm:PinSocket_2x20_P2.54mm_Vertical -> Wsprry Pi:PinSocket_2x20_P2.54mm_Vertical; symbol Connector_Generic:Conn_02x20_Odd_Even -> Wsprry Pi:Conn_02x20_Odd_Even
- J81, J82: footprint Connector_PinSocket_2.54mm:PinSocket_1x04_P2.54mm_Vertical -> Wsprry Pi:PinSocket_1x04_P2.54mm_Vertical; symbol Connector_Generic:Conn_01x04 -> Wsprry Pi:Conn_01x04
- R11, R41, R42, R43: footprint Resistor_SMD:R_0603_1608Metric -> Wsprry Pi:R_0603_1608Metric; symbol Device:R_US -> Wsprry Pi:R_US
- R21, R31, R32: footprint Resistor_SMD:R_0402_1005Metric -> Wsprry Pi:R_0402_1005Metric; symbol Device:R_US -> Wsprry Pi:R_US
- R51: footprint Resistor_SMD:R_0805_2012Metric -> Wsprry Pi:R_0805_2012Metric; symbol Device:R_US -> Wsprry Pi:R_US
- U51: footprint Package_TO_SOT_SMD:SOT-89-3 -> Wsprry Pi:SOT-89-3; symbol RF_Amplifier:GVA-84 -> Wsprry Pi:GVA-84
- Y21: footprint Oscillator:Oscillator_SMD_SeikoEpson_TG2520SMN-xxx-xxxxxx-4Pin_2.5x2.0mm -> Wsprry Pi:Oscillator_SMD_SeikoEpson_TG2520SMN-xxx-xxxxxx-4Pin_2.5x2.0mm; symbol Oscillator:TG2520SMN-xx.xxxxxxMhz-xxxxNM -> Wsprry Pi:TG2520SMN-xx.xxxxxxMhz-xxxxNM
- Y31: footprint Package_SO:MSOP-10_3x3mm_P0.5mm -> Wsprry Pi:MSOP-10_3x3mm_P0.5mm; symbol Oscillator:Si5351A-B-GT -> Wsprry Pi:Si5351A-B-GT
