File: Wsprry-Pi-LPF/Wsprry-Pi-LPF.kicad_sch (KiCad schematic)
At the start: 13 parts, among them J1 Conn_01x04, J2 Conn_01x04

Commit message: Cleanup due to lost libraries
Parts:
- CA1, CA3, CA5, CA7, CB1, CB3, CB5, CB7: footprint Capacitor_THT:C_Disc_D3.0mm_W1.6mm_P2.50mm -> Wsprry Pi LPF:C_Disc_D3.0mm_W1.6mm_P2.50mm; symbol Device:C -> Wsprry Pi LPF:C
- J1, J2: footprint Connector_PinHeader_2.54mm:PinHeader_1x04_P2.54mm_Vertical -> Wsprry Pi LPF:PinHeader_1x04_P2.54mm_Vertical; symbol Connector_Generic:Conn_01x04 -> Wsprry Pi LPF:Conn_01x04
- L2, L4, L6: symbol Device:L -> Wsprry Pi LPF:L
Changed lines of the file:
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@@
 	)
 	(symbol
-		(lib_id "power:GND")
+		(lib_id "Wsprry Pi LPF:GND")
 		(at 196.85 102.87 180)
 		(unit 1)
@@
 	)
 	(symbol
-		(lib_id "Device:C")
+		(lib_id "Wsprry Pi LPF:C")
 		(at 186.69 95.25 0)
 		(unit 1)
@@
 			)
 		)
-		(property "Footprint" "Capacitor_THT:C_Disc_D3.0mm_W1.6mm_P2.50mm"
+		(property "Footprint" "Wsprry Pi LPF:C_Disc_D3.0mm_W1.6mm_P2.50mm"
 			(at 187.6552 99.06 0)
 			(effects
@@
 	)
 	(symbol
-		(lib_id "Device:C")
+		(lib_id "Wsprry Pi LPF:C")
 		(at 156.21 95.25 0)
 		(unit 1)
@@
 			)
 		)
-		(property "Footprint" "Capacitor_THT:C_Disc_D3.0mm_W1.6mm_P2.50mm"
+		(property "Footprint" "Wsprry Pi LPF:C_Disc_D3.0mm_W1.6mm_P2.50mm"
 			(at 157.1752 99.06 0)
 			(effects
@@
 	)
 	(symbol
-		(lib_id "Device:C")
+		(lib_id "Wsprry Pi LPF:C")
 		(at 115.57 95.25 0)
 		(unit 1)
@@
 			)
 		)
-		(property "Footprint" "Capacitor_THT:C_Disc_D3.0mm_W1.6mm_P2.50mm"
+		(property "Footprint" "Wsprry Pi LPF:C_Disc_D3.0mm_W1.6mm_P2.50mm"
 			(at 116.5352 99.06 0)
 			(effects
@@
 	)
 	(symbol
-		(lib_id "Device:L")
+		(lib_id "Wsprry Pi LPF:L")
 		(at 171.45 107.95 0)
 		(unit 1)
@@
 	)
 	(symbol
-		(lib_id "Device:C")
+		(lib_id "Wsprry Pi LPF:C")
 		(at 135.89 95.25 0)
 		(unit 1)
@@
 			)
 		)
-		(property "Footprint" "Capacitor_THT:C_Disc_D3.0mm_W1.6mm_P2.50mm"
+		(property "Footprint" "Wsprry Pi LPF:C_Disc_D3.0mm_W1.6mm_P2.50mm"
 			(at 136.8552 99.06 0)
 			(effects
@@
 	)
 	(symbol
-		(lib_id "Device:L")
+		(lib_id "Wsprry Pi LPF:L")
 		(at 130.81 107.95 0)
 		(unit 1)
@@
 	)
 	(symbol
-		(lib_id "power:GND")
+		(lib_id "Wsprry Pi LPF:GND")
 		(at 120.65 88.9 180)
 		(unit 1)
@@
 	)
 	(symbol
-		(lib_id "Device:C")
+		(lib_id "Wsprry Pi LPF:C")
 		(at 146.05 95.25 0)
 		(unit 1)
@@
 			)
 		)
-		(property "Footprint" "Capacitor_THT:C_Disc_D3.0mm_W1.6mm_P2.50mm"
+		(property "Footprint" "Wsprry Pi LPF:C_Disc_D3.0mm_W1.6mm_P2.50mm"
 			(at 147.0152 99.06 0)
 			(effects
@@
 	)
 	(symbol
-		(lib_id "Device:C")
+		(lib_id "Wsprry Pi LPF:C")
 		(at 176.53 95.25 0)
 		(unit 1)
@@
 			)
 		)
-		(property "Footprint" "Capacitor_THT:C_Disc_D3.0mm_W1.6mm_P2.50mm"
+		(property "Footprint" "Wsprry Pi LPF:C_Disc_D3.0mm_W1.6mm_P2.50mm"
 			(at 177.4952 99.06 0)
 			(effects
@@
 	)
 	(symbol
-		(lib_id "Connector_Generic:Conn_01x04")
+		(lib_id "Wsprry Pi LPF:Conn_01x04")
 		(at 190.5 106.68 0)
 		(mirror y)
@@
 			)
 		)
-		(property "Footprint" "Connector_PinHeader_2.54mm:PinHeader_1x04_P2.54mm_Vertical"
+		(property "Footprint" "Wsprry Pi LPF:PinHeader_1x04_P2.54mm_Vertical"
 			(at 190.5 106.68 0)
 			(effects
@@
 	)
 	(symbol
-		(lib_id "power:GND")
+		(lib_id "Wsprry Pi LPF:GND")
 		(at 181.61 88.9 180)
 		(unit 1)
@@
 	)
 	(symbol
-		(lib_id "power:GND")
+		(lib_id "Wsprry Pi LPF:GND")
 		(at 105.41 113.03 0)
 		(unit 1)
@@
 	)
 	(symbol
-		(lib_id "power:GND")
+		(lib_id "Wsprry Pi LPF:GND")
 		(at 196.85 113.03 0)
 		(unit 1)
@@
 	)
 	(symbol
-		(lib_id "Connector_Generic:Conn_01x04")
+		(lib_id "Wsprry Pi LPF:Conn_01x04")
 		(at 111.76 106.68 0)
 		(unit 1)
@@
 			)
 		)
-		(property "Footprint" "Connector_PinHeader_2.54mm:PinHeader_1x04_P2.54mm_Vertical"
+		(property "Footprint" "Wsprry Pi LPF:PinHeader_1x04_P2.54mm_Vertical"
 			(at 111.76 106.68 0)
 			(effects
@@
 	)
 	(symbol
-		(lib_id "power:GND")
+		(lib_id "Wsprry Pi LPF:GND")
 		(at 105.41 102.87 180)
 		(unit 1)
@@
 	)
 	(symbol
-		(lib_id "power:GND")
+		(lib_id "Wsprry Pi LPF:GND")
 		(at 161.29 88.9 180)
 		(unit 1)
@@
 	)
 	(symbol
-		(lib_id "Device:C")
+		(lib_id "Wsprry Pi LPF:C")
 		(at 125.73 95.25 0)
 		(unit 1)
@@
 			)
 		)
-		(property "Footprint" "Capacitor_THT:C_Disc_D3.0mm_W1.6mm_P2.50mm"
+		(property "Footprint" "Wsprry Pi LPF:C_Disc_D3.0mm_W1.6mm_P2.50mm"
 			(at 126.6952 99.06 0)
 			(effects
@@
 	)
 	(symbol
-		(lib_id "power:GND")
+		(lib_id "Wsprry Pi LPF:GND")
 		(at 140.97 88.9 180)
 		(unit 1)
@@
 	)
 	(symbol
-		(lib_id "Device:L")
+		(lib_id "Wsprry Pi LPF:L")
 		(at 151.13 107.95 0)
 		(unit 1)
@@
 	)
 	(symbol
-		(lib_id "Device:C")
+		(lib_id "Wsprry Pi LPF:C")
 		(at 166.37 95.25 0)
 		(unit 1)
@@
 			)
 		)
-		(property "Footprint" "Capacitor_THT:C_Disc_D3.0mm_W1.6mm_P2.50mm"
+		(property "Footprint" "Wsprry Pi LPF:C_Disc_D3.0mm_W1.6mm_P2.50mm"
 			(at 167.3352 99.06 0)
 			(effects

Commit message: Update LPF KiCad version and exclude hand-fitted headers from BOM
Parts:
- J1, J2: LCSC C2718488 -> (none); LCSC_PART C2718488 -> (none); now left out of the parts list
