File: Wsprry-Pi-GPIO-Univ/Wsprry-Pi-GPIO-Univ.kicad_sch (KiCad schematic)
At the start: 21 parts, among them J11 GPIO, J81 Conn_01x04, J82 Conn_01x04, J83 SMA, SW11 Switch, U51 GVA-84

Commit message: Cleanup due to lost libraries
Parts:
- C12, C51: footprint Capacitor_SMD:C_0603_1608Metric -> Wsprry Pi:C_0603_1608Metric; symbol Device:C -> Wsprry Pi:C
- C52, C53: footprint Capacitor_SMD:C_0402_1005Metric -> Wsprry Pi:C_0402_1005Metric; symbol Device:C -> Wsprry Pi:C
- C54, C55: footprint Capacitor_SMD:C_0805_2012Metric -> Wsprry Pi:C_0805_2012Metric; symbol Device:C -> Wsprry Pi:C
- D11: footprint LED_SMD:LED_0603_1608Metric -> Wsprry Pi:LED_0603_1608Metric; symbol Device:LED -> Wsprry Pi:LED
- FB11, FB51: footprint Inductor_SMD:L_0603_1608Metric -> Wsprry Pi:L_0603_1608Metric; symbol Device:FerriteBead -> Wsprry Pi:FerriteBead
- J11: footprint Connector_PinSocket_2.54mm:PinSocket_2x20_P2.54mm_Vertical -> Wsprry Pi:PinSocket_2x20_P2.54mm_Vertical; symbol Connector_Generic:Conn_02x20_Odd_Even -> Wsprry Pi:Conn_02x20_Odd_Even
- J81, J82: footprint Connector_PinSocket_2.54mm:PinSocket_1x04_P2.54mm_Vertical -> Wsprry Pi:PinSocket_1x04_P2.54mm_Vertical; symbol Connector_Generic:Conn_01x04 -> Wsprry Pi:Conn_01x04
- R11, R41, R42, R43: footprint Resistor_SMD:R_0603_1608Metric -> Wsprry Pi:R_0603_1608Metric; symbol Device:R_US -> Wsprry Pi:R_US
- R51: footprint Resistor_SMD:R_0805_2012Metric -> Wsprry Pi:R_0805_2012Metric; symbol Device:R_US -> Wsprry Pi:R_US
- U51: footprint Package_TO_SOT_SMD:SOT-89-3 -> Wsprry Pi:SOT-89-3; symbol RF_Amplifier:GVA-84 -> Wsprry Pi:GVA-84
Changed lines of the file:
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@@
 	)
 	(symbol
-		(lib_id "Device:FerriteBead")
+		(lib_id "Wsprry Pi:FerriteBead")
 		(at 205.74 73.66 90)
 		(unit 1)
@@
 			)
 		)
-		(property "Footprint" "Inductor_SMD:L_0603_1608Metric"
+		(property "Footprint" "Wsprry Pi:L_0603_1608Metric"
 			(at 205.74 75.438 90)
 			(effects
@@
 	)
 	(symbol
-		(lib_id "Device:C")
+		(lib_id "Wsprry Pi:C")
 		(at 228.6 68.58 180)
 		(unit 1)
@@
 			)
 		)
-		(property "Footprint" "Capacitor_SMD:C_0402_1005Metric"
+		(property "Footprint" "Wsprry Pi:C_0402_1005Metric"
 			(at 227.6348 64.77 0)
 			(effects
@@
 	)
 	(symbol
-		(lib_id "power:GND")
+		(lib_id "Wsprry Pi:GND")
 		(at 31.75 176.53 180)
 		(unit 1)
@@
 	)
 	(symbol
-		(lib_id "Device:R_US")
+		(lib_id "Wsprry Pi:R_US")
 		(at 73.66 53.34 270)
 		(unit 1)
@@
 			)
 		)
-		(property "Footprint" "Resistor_SMD:R_0603_1608Metric"
+		(property "Footprint" "Wsprry Pi:R_0603_1608Metric"
 			(at 73.406 54.356 90)
 			(effects
@@
 	)
 	(symbol
-		(lib_id "Device:R_US")
+		(lib_id "Wsprry Pi:R_US")
 		(at 219.71 29.21 90)
 		(unit 1)
@@
 			)
 		)
-		(property "Footprint" "Resistor_SMD:R_0603_1608Metric"
+		(property "Footprint" "Wsprry Pi:R_0603_1608Metric"
 			(at 219.964 28.194 90)
 			(effects
@@
 	)
 	(symbol
-		(lib_id "Device:C")
+		(lib_id "Wsprry Pi:C")
 		(at 80.01 35.56 0)
 		(mirror x)
@@
 			)
 		)
-		(property "Footprint" "Capacitor_SMD:C_0603_1608Metric"
+		(property "Footprint" "Wsprry Pi:C_0603_1608Metric"
 			(at 80.9752 31.75 0)
 			(effects
@@
 	)
 	(symbol
-		(lib_id "Device:C")
+		(lib_id "Wsprry Pi:C")
 		(at 247.65 87.63 90)
 		(unit 1)
@@
 			)
 		)
-		(property "Footprint" "Capacitor_SMD:C_0805_2012Metric"
+		(property "Footprint" "Wsprry Pi:C_0805_2012Metric"
 			(at 251.46 86.6648 0)
 			(effects
@@
 	)
 	(symbol
-		(lib_id "power:GND")
+		(lib_id "Wsprry Pi:GND")
 		(at 217.17 96.52 0)
 		(unit 1)
@@
 	)
 	(symbol
-		(lib_id "power:GND")
+		(lib_id "Wsprry Pi:GND")
 		(at 78.74 53.34 90)
 		(unit 1)
@@
 	)
 	(symbol
-		(lib_id "power:PWR_FLAG")
+		(lib_id "Wsprry Pi:PWR_FLAG")
 		(at 59.69 40.64 0)
 		(unit 1)
@@
 	)
 	(symbol
-		(lib_id "Connector_Generic:Conn_02x20_Odd_Even")
+		(lib_id "Wsprry Pi:Conn_02x20_Odd_Even")
 		(at 49.53 63.5 0)
 		(unit 1)
@@
 			)
 		)
-		(property "Footprint" "Connector_PinSocket_2.54mm:PinSocket_2x20_P2.54mm_Vertical"
+		(property "Footprint" "Wsprry Pi:PinSocket_2x20_P2.54mm_Vertical"
 			(at -73.66 87.63 0)
 			(effects
@@
 	)
 	(symbol
-		(lib_id "power:PWR_FLAG")
+		(lib_id "Wsprry Pi:PWR_FLAG")
 		(at 41.91 91.44 270)
 		(unit 1)
@@
 	)
 	(symbol
-		(lib_id "power:GND")
+		(lib_id "Wsprry Pi:GND")
 		(at 210.82 63.5 180)
 		(unit 1)
@@
 	)
 	(symbol
-		(lib_id "Device:R_US")
+		(lib_id "Wsprry Pi:R_US")
 		(at 209.55 29.21 90)
 		(unit 1)
@@
 			)
 		)
-		(property "Footprint" "Resistor_SMD:R_0603_1608Metric"
+		(property "Footprint" "Wsprry Pi:R_0603_1608Metric"
 			(at 209.804 28.194 90)
 			(effects
@@
 	)
 	(symbol
-		(lib_id "Device:R_US")
+		(lib_id "Wsprry Pi:R_US")
 		(at 228.6 81.28 0)
 		(unit 1)
@@
 			)
 		)
-		(property "Footprint" "Resistor_SMD:R_0805_2012Metric"
+		(property "Footprint" "Wsprry Pi:R_0805_2012Metric"
 			(at 229.616 81.534 90)
 			(effects
@@
 	)
 	(symbol
-		(lib_id "power:GND")
+		(lib_id "Wsprry Pi:GND")
 		(at 67.31 191.77 0)
 		(unit 1)
@@
 	)
 	(symbol
-		(lib_id "Device:FerriteBead")
+		(lib_id "Wsprry Pi:FerriteBead")
 		(at 63.5 40.64 90)
 		(mirror x)
@@
 			)
 		)
-		(property "Footprint" "Inductor_SMD:L_0603_1608Metric"
+		(property "Footprint" "Wsprry Pi:L_0603_1608Metric"
 			(at 63.5 38.862 90)
 			(effects
@@
 	)
 	(symbol
-		(lib_id "Device:R_US")
+		(lib_id "Wsprry Pi:R_US")
 		(at 214.63 34.29 180)
 		(unit 1)
@@
 			)
 		)
-		(property "Footprint" "Resistor_SMD:R_0603_1608Metric"
+		(property "Footprint" "Wsprry Pi:R_0603_1608Metric"
 			(at 213.614 34.036 90)
 			(effects
@@
 	)
 	(symbol
-		(lib_id "power:GND")
+		(lib_id "Wsprry Pi:GND")
 		(at 46.99 176.53 180)
 		(unit 1)
@@
 	)
 	(symbol
-		(lib_id "Device:C")
+		(lib_id "Wsprry Pi:C")
 		(at 219.71 68.58 180)
 		(unit 1)
@@
 			)
 		)
-		(property "Footprint" "Capacitor_SMD:C_0402_1005Metric"
+		(property "Footprint" "Wsprry Pi:C_0402_1005Metric"
 			(at 218.7448 64.77 0)
 			(effects
@@
 	)
 	(symbol
-		(lib_id "power:GND")
+		(lib_id "Wsprry Pi:GND")
 		(at 46.99 186.69 0)
 		(unit 1)
@@
 	)
 	(symbol
-		(lib_id "power:GND")
+		(lib_id "Wsprry Pi:GND")
 		(at 41.91 92.71 0)
 		(unit 1)
@@
 	)
 	(symbol
-		(lib_id "Connector_Generic:Conn_01x04")
+		(lib_id "Wsprry Pi:Conn_01x04")
 		(at 41.91 180.34 0)
 		(mirror y)
@@
 			)
 		)
-		(property "Footprint" "Connector_PinSocket_2.54mm:PinSocket_1x04_P2.54mm_Vertical"
+		(property "Footprint" "Wsprry Pi:PinSocket_1x04_P2.54mm_Vertical"
 			(at 41.91 180.34 0)
 			(effects
@@
 	)
 	(symbol
-		(lib_id "power:GND")
+		(lib_id "Wsprry Pi:GND")
 		(at 80.01 27.94 0)
 		(mirror x)
@@
 	)
 	(symbol
-		(lib_id "power:GND")
+		(lib_id "Wsprry Pi:GND")
 		(at 59.69 92.71 0)
 		(unit 1)
@@
 	)
 	(symbol
-		(lib_id "power:GND")
+		(lib_id "Wsprry Pi:GND")
 		(at 214.63 39.37 0)
 		(unit 1)
@@
 	)
 	(symbol
-		(lib_id "power:GND")
+		(lib_id "Wsprry Pi:GND")
 		(at 22.86 85.09 0)
 		(unit 1)
@@
 	)
 	(symbol
-		(lib_id "Device:LED")
+		(lib_id "Wsprry Pi:LED")
 		(at 64.77 53.34 180)
 		(unit 1)
@@
 			)
 		)
-		(property "Footprint" "LED_SMD:LED_0603_1608Metric"
+		(property "Footprint" "Wsprry Pi:LED_0603_1608Metric"
 			(at 64.77 53.34 0)
 			(effects
@@
 	)
 	(symbol
-		(lib_id "Connector_Generic:Conn_01x04")
+		(lib_id "Wsprry Pi:Conn_01x04")
 		(at 36.83 180.34 0)
 		(unit 1)
@@
 			)
 		)
-		(property "Footprint" "Connector_PinSocket_2.54mm:PinSocket_1x04_P2.54mm_Vertical"
+		(property "Footprint" "Wsprry Pi:PinSocket_1x04_P2.54mm_Vertical"
 			(at 36.83 180.34 0)
 			(effects
@@
 	)
 	(symbol
-		(lib_id "RF_Amplifier:GVA-84")
+		(lib_id "Wsprry Pi:GVA-84")
 		(at 219.71 87.63 0)
 		(unit 1)
@@
 			)
 		)
-		(property "Footprint" "Package_TO_SOT_SMD:SOT-89-3"
+		(property "Footprint" "Wsprry Pi:SOT-89-3"
 			(at 220.98 77.47 0)
 			(effects
@@
 	)
 	(symbol
-		(lib_id "power:GND")
+		(lib_id "Wsprry Pi:GND")
 		(at 31.75 186.69 0)
 		(unit 1)
@@
 	)
 	(symbol
-		(lib_id "power:GND")
+		(lib_id "Wsprry Pi:GND")
 		(at 68.58 27.94 0)
 		(mirror x)
@@
 	)
 	(symbol
-		(lib_id "power:PWR_FLAG")
+		(lib_id "Wsprry Pi:PWR_FLAG")
 		(at 40.64 60.96 180)
 		(unit 1)
@@
 	)
 	(symbol
-		(lib_id "Device:C")
+		(lib_id "Wsprry Pi:C")
 		(at 199.39 87.63 90)
 		(unit 1)
@@
 			)
 		)
-		(property "Footprint" "Capacitor_SMD:C_0805_2012Metric"
+		(property "Footprint" "Wsprry Pi:C_0805_2012Metric"
 			(at 203.2 86.6648 0)
 			(effects
@@
 	)
 	(symbol
-		(lib_id "Device:C")
+		(lib_id "Wsprry Pi:C")
 		(at 210.82 68.58 180)
 		(unit 1)
@@
 			)
 		)
-		(property "Footprint" "Capacitor_SMD:C_0603_1608Metric"
+		(property "Footprint" "Wsprry Pi:C_0603_1608Metric"
 			(at 209.8548 64.77 0)
 			(effects
@@
 	)
 	(symbol
-		(lib_id "power:GND")
+		(lib_id "Wsprry Pi:GND")
 		(at 219.71 63.5 180)
 		(unit 1)
@@
 	)
 	(symbol
-		(lib_id "power:GND")
+		(lib_id "Wsprry Pi:GND")
 		(at 228.6 63.5 180)
 		(unit 1)

Commit message: Add GPIO Selector
Parts:
- added J21: GPIO Select, Connector_PinHeader_1.00mm:PinHeader_1x03_P1.00mm_Vertical, symbol Connector_Generic:Conn_01x03
Connections:
- net GPIO_CLK: now also J21.2 (Pin_2); no longer J11.7 (Pin_7)
- net GPIO_CLK20: now reaches J11.38 (Pin_38)
- net GPIO_CLK20: now also J21.3 (Pin_3)
- new net GPIO_CLK4: J11.7 (Pin_7), J21.1 (Pin_1)
- no-connect marks 26 -> 25

Commit message: Re-purpose for broadband amp
Parts:
- removed C51: 1µF, Wsprry Pi:C_0603_1608Metric, symbol Wsprry Pi:C
- removed C52: 100nF, Wsprry Pi:C_0402_1005Metric, symbol Wsprry Pi:C
- removed C53: 10nF, Wsprry Pi:C_0402_1005Metric, symbol Wsprry Pi:C
- removed C54, C55: 1uF, Wsprry Pi:C_0805_2012Metric, symbol Wsprry Pi:C
- removed FB51: 600Ω@100MHz, Wsprry Pi:L_0603_1608Metric, symbol Wsprry Pi:FerriteBead
- removed R41, R43: 40.2Ω, Wsprry Pi:R_0603_1608Metric, symbol Wsprry Pi:R_US
- removed R42: 10Ω, Wsprry Pi:R_0603_1608Metric, symbol Wsprry Pi:R_US
- removed R51: 10Ω, Wsprry Pi:R_0805_2012Metric, symbol Wsprry Pi:R_US
- removed U51: GVA-84, Wsprry Pi:SOT-89-3, symbol Wsprry Pi:GVA-84
- C11: value 100µF -> 47µF
- J11, J21, J81, J82: now left out of the parts list
- J83: value SMA -> SMA_Adafruit_1865; footprint Wsprry Pi:SMA-TH_BWSMA-KWE-Z001 -> Wsprry Pi:SMA_Adafruit_1865_EdgeMount; symbol Wsprry Pi:BWSMA-KWE-Z001 -> Wsprry Pi:SMA_Adafruit_1865; LCSC C496551 -> (none); LCSC Part Name 内孔 SMA 弯头 -> (none); LCSC_PART C496551 -> (none); MPN (none) -> 1865; Manufacturer BAT WIRELESS(蝙蝠无线) -> Adafruit; Manufacturer Part BWSMA-KWE-Z001 -> (none); Supplier LCSC -> (none); Supplier Part C496551 -> (none); now left out of the parts list
Connections:
- net GND: no longer J83.1, J83.3, J83.4
- net RF_OUT: now also J83.1 (In); no longer J83.5
Other:
- moved on the sheet: C11, C12, D11, FB11, J11, J21, J81, J82, R11, SW11
