File: WsprryPi-GPIO-Univ/WsprryPi-GPIO-Univ.kicad_pcb (KiCad board)
At the start: 2 copper layers, 65 x 30 mm, 15 parts, among them J11 GPIO, J21 GPIO Select, J81 Conn_01x04, J82 Conn_01x04, J83 SMA_Adafruit_1865, SW11 Switch

Commit message: Rename GPIO project and document amplifier requirements
Parts:
- removed C11: 47µF, Wsprry Pi:CAP-SMD_BD6.3-L6.6-W6.6-FD
- removed C12: 100nF, Wsprry Pi:C_0603_1608Metric
- removed FB11: 600Ω@100MHz, Wsprry Pi:L_0603_1608Metric
Routing:
- net /5V_RAIL: track 37.2 -> 0.00 mm
- net GND: track 30.5 -> 17.3 mm, vias 297 -> 222
- net /5V: track 9.09 -> 8.00 mm

Commit message: Import amplifier input parts and update GPIO selector layout
Parts:
- moved J21 19.1 mm to (121.0, 79.0)
Routing:
- net /GPIO_CLK20: track 16.2 -> 35.6 mm
- net /GPIO_CLK4: track 26.5 -> 7.77 mm

Commit message: Add GPIO broadband amplifier schematic blocks
Add the PA, bipolar supply, and protected Pi power-input circuitry, along with project-local symbols, footprints, and available STEP models. Localize all placed schematic symbols and assigned footprints.
Parts:
- J21: footprint Connector_PinHeader_1.00mm:PinHeader_1x03_P1.00mm_Vertical -> Wsprry Pi:PinHeader_1x03_P1.00mm_Vertical
Changed lines of the file:
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@@
 		(embedded_fonts no)
 	)
-	(footprint "Connector_PinHeader_1.00mm:PinHeader_1x03_P1.00mm_Vertical"
+	(footprint "Wsprry Pi:PinHeader_1x03_P1.00mm_Vertical"
 		(layer "F.Cu")
 		(at 120.99 79 90)
@@
 		)
 		(embedded_fonts no)
-		(model "${KICAD10_3DMODEL_DIR}/Connector_PinHeader_1.00mm.3dshapes/PinHeader_1x03_P1.00mm_Vertical.step"
+		(model "${KIPRJMOD}/libraries/3dmodels/Connector_PinHeader_1.00mm.3dshapes/PinHeader_1x03_P1.00mm_Vertical.step"
 			(offset
 				(xyz 0 0 0)
