File: WsprryPi Zero GPIO/WsprryPi Zero GPIO.kicad_sch (KiCad schematic)
At the start: 28 parts, among them J1 SMA_Adafruit_1865, J11 Socket_2x20_P2.54mm, J12 Conn_01x03, J41 J81/J82 LPF sockets, SW11 SKRPANE010, T22 YA9308-AEC, T40 YA9308-AEC, U10 Raspberry Pi 40-pin HAT inter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, U32 LTC6432AIUF-15#PBF, U50 TPS22918DBVR

Commit message: Update cap type
Parts:
- removed C30, C36: 1µF, wsprrypi-zero-gpio:C_0805_2012Metric, symbol wsprrypi-zero-gpio:C_0805
- added C34: 1µF, wsprrypi-zero-gpio:C_0805_2012Metric, symbol wsprrypi-zero-gpio:C_0805
- added C38: 1µF, wsprrypi-zero-gpio:C_1206_3216Metric, symbol wsprrypi-zero-gpio:C_0805
- C21, C31, C32, C37: footprint wsprrypi-zero-gpio:C_0805_2012Metric -> wsprrypi-zero-gpio:C_1206_3216Metric; LCSC_PART C28323 -> C342628
- renumbered C34 to C35, C35 to C36, C53 to C52, C55 to C53, J1 to J41, J41 to J42, R20 to R21, R21 to R22, R52 to R51, R54 to R52, T22 to T21, T40 to T41, U10 to U11, U32 to U31, U50 to U51
Connections:
- net AMP_OUT_N: now also C37.2
- net AMP_OUT_P: now also C38.2; no longer C37.2
- net GND: now also C34.1; no longer C32.1
- net RF_DIFF_N: now also C31.1
- net RF_DIFF_P: now also C32.1; no longer C31.1
- net at U31.12 (-FDBK): now also C37.1
- net at U31.19 (+FDBK): now also C38.1; no longer C37.1
- net at U31.24 (+IN): now also C32.2; no longer C31.2
- net at U31.5 (NFILT2): now also C33.2; no longer C32.2
- net at U31.6 (NFILT1): now also C34.2; no longer C33.2
- net at U31.7 (-IN): now also C31.2

Commit message: Swap transformer
Parts:
- removed T21, T41: YA9308-AEC, wsprrypi-zero-gpio:Coilcraft_YA9308, symbol wsprrypi-zero-gpio:YA9308-AEC
- added T21, T41: WBC2-1TLC, wsprrypi-zero-gpio:Coilcraft_WBC2-1TLC, symbol wsprrypi-zero-gpio:WBC2-1TLC
Connections:
- net AMP_OUT_N: now also T41.1 (SEC1)
- net AMP_OUT_P: now also T41.3 (SEC2)
- net GND: now also T21.4 (PRI2), T41.4 (PRI2)
- net RF_DIFF_N: now also T21.1 (SEC1)
- net RF_DIFF_P: now also T21.3 (SEC2)
- net SW_5V: now also T41.2 (CT)
- net TX_OUT: now also T41.6 (PRI1)
- net at C21.2, R22.2: now also T21.6 (PRI1)
- no-connect marks 27 -> 28
Changed lines of the file:
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@@
 	)
 	(no_connect
+		(at 245.11 100.33)
+	)
+	(no_connect
 		(at 24.13 54.61)
 	)
@@
 	)
 	(symbol
-		(lib_id "wsprrypi-zero-gpio:YA9308-AEC")
-		(at 236.22 100.33 180)
+		(lib_id "wsprrypi-zero-gpio:WBC2-1TLC")
+		(at 130.81 30.48 0)
 		(unit 1)
 		(body_style 1)
@@
 		(in_pos_files yes)
 		(dnp no)
-		(property "Reference" "T41"
-			(at 235.712 105.41 0)
+		(property "Reference" "T21"
+			(at 130.81 30.48 0)
 			(show_name no)
 			(do_not_autoplace no)
@@
 			)
 		)
-		(property "Value" "YA9308-AEC"
-			(at 236.22 92.202 0)
+		(property "Value" "WBC2-1TLC"
+			(at 130.81 22.86 0)
 			(show_name no)
 			(do_not_autoplace no)
@@
 			)
 		)
-		(property "Footprint" "wsprrypi-zero-gpio:Coilcraft_YA9308"
-			(at 237.45 94.15 0)
+		(property "Footprint" "wsprrypi-zero-gpio:Coilcraft_WBC2-1TLC"
+			(at 130.81 30.48 0)
 			(hide yes)
 			(show_name no)
@@
 			)
 		)
-		(property "Datasheet" "https://www.coilcraft.com/getmedia/508634a8-8a9d-4933-83b8-7660d3e9ca71/ya9308.pdf"
-			(at 237.45 94.15 0)
+		(property "Datasheet" "https://www.coilcraft.com/getmedia/f685d903-2563-4c96-8ba6-f82a58883aeb/wbc.pdf"
+			(at 130.81 30.48 0)
 			(hide yes)
 			(show_name no)
@@
 			)
 		)
-		(property "Description" "1:2 impedance-ratio SMT wideband transformer, 0.1 MHz to 950 MHz, center-tapped secondary"
-			(at 237.45 94.15 0)
+		(property "Description" "1:2 impedance-ratio SMT wideband transformer, 0.2 MHz to 500 MHz, center-tapped secondary"
+			(at 130.81 30.48 0)
 			(hide yes)
 			(show_name no)
@@
 		)
 		(property "Manufacturer" "Coilcraft"
-			(at 237.45 94.15 0)
+			(at 130.81 30.48 0)
 			(hide yes)
 			(show_name no)
@@
 			)
 		)
-		(property "MPN" "YA9308-AEC"
-			(at 237.45 94.15 0)
+		(property "MPN" "WBC2-1TLC"
+			(at 130.81 30.48 0)
 			(hide yes)
 			(show_name no)
@@
 			)
 		)
-		(pin "1"
+		(property "LCSC_PART" "C19191658"
+			(at 130.81 30.48 0)
+			(hide yes)
+			(show_name no)
+			(do_not_autoplace no)
+			(effects
+				(font
+					(size 1.27 1.27)
+				)
+			)
+		)
+		(pin "5"
 		)
 		(pin "2"
@@
 		(pin "3"
 		)
-		(pin "4"
-		)
-		(pin "5"
+		(pin "1"
 		)
 		(pin "6"
 		)
+		(pin "4"
+		)
 		(instances
 			(project "WsprryPi Zero GPIO"
 				(path "/42fb2efa-c288-4686-a90a-043ad23a327d"
-					(reference "T41")
+					(reference "T21")
 					(unit 1)
 				)
@@
 	)
 	(symbol
-		(lib_id "wsprrypi-zero-gpio:YA9308-AEC")
-		(at 130.81 30.48 0)
-		(unit 1)
-		(body_style 1)
-		(exclude_from_sim no)
-		(in_bom yes)
-		(on_board yes)
-		(in_pos_files yes)
-		(dnp no)
-		(property "Reference" "T21"
-			(at 130.556 25.908 0)
-			(show_name no)
-			(do_not_autoplace no)
-			(effects
-				(font
-					(size 1.27 1.27)
-				)
-			)
-		)
-		(property "Value" "YA9308-AEC"
-			(at 130.556 23.114 0)
-			(show_name no)
-			(do_not_autoplace no)
-			(effects
-				(font
-					(size 1.27 1.27)
-				)
-			)
-		)
-		(property "Footprint" "wsprrypi-zero-gpio:Coilcraft_YA9308"
-			(at 131.03 36.66 0)
-			(hide yes)
-			(show_name no)
-			(do_not_autoplace no)
-			(effects
-				(font
-					(size 1.27 1.27)
-				)
-			)
-		)
-		(property "Datasheet" "https://www.coilcraft.com/getmedia/508634a8-8a9d-4933-83b8-7660d3e9ca71/ya9308.pdf"
-			(at 131.03 36.66 0)
-			(hide yes)
-			(show_name no)
-			(do_not_autoplace no)
-			(effects
-				(font
-					(size 1.27 1.27)
-				)
-			)
-		)
-		(property "Description" "1:2 impedance-ratio SMT wideband transformer, 0.1 MHz to 950 MHz, center-tapped secondary"
-			(at 131.03 36.66 0)
-			(hide yes)
-			(show_name no)
-			(do_not_autoplace no)
-			(effects
-				(font
-					(size 1.27 1.27)
-				)
-			)
-		)
-		(property "Manufacturer" "Coilcraft"
-			(at 131.03 36.66 0)
-			(hide yes)
-			(show_name no)
-			(do_not_autoplace no)
-			(effects
-				(font
-					(size 1.27 1.27)
-				)
-			)
-		)
-		(property "MPN" "YA9308-AEC"
-			(at 131.03 36.66 0)
-			(hide yes)
-			(show_name no)
-			(do_not_autoplace no)
-			(effects
-				(font
-					(size 1.27 1.27)
-				)
-			)
-		)
-		(pin "1"
-		)
-		(pin "2"
-		)
-		(pin "3"
-		)
-		(pin "4"
-		)
-		(pin "5"
-		)
-		(pin "6"
-		)
-		(instances
-			(project "WsprryPi Zero GPIO"
-				(path "/42fb2efa-c288-4686-a90a-043ad23a327d"
-					(reference "T21")
-					(unit 1)
-				)
-			)
-		)
-	)
-	(symbol
 		(lib_id "wsprrypi-zero-gpio:GND")
 		(at 91.44 80.01 0)
@@
 					(unit 1)
 				)
+			)
+		)
+	)
+	(symbol
+		(lib_id "wsprrypi-zero-gpio:WBC2-1TLC")
+		(at 236.22 100.33 180)
+		(unit 1)
+		(body_style 1)
+		(exclude_from_sim no)
+		(in_bom yes)
+		(on_board yes)
+		(in_pos_files yes)
+		(dnp no)
+		(property "Reference" "T41"
+			(at 236.22 100.584 0)
+			(show_name no)
+			(do_not_autoplace no)
+			(effects
+				(font
+					(size 1.27 1.27)
+				)
+			)
+		)
+		(property "Value" "WBC2-1TLC"
+			(at 236.22 92.71 0)
+			(show_name no)
+			(do_not_autoplace no)
+			(effects
+				(font
+					(size 1.27 1.27)
+				)
+			)
+		)
+		(property "Footprint" "wsprrypi-zero-gpio:Coilcraft_WBC2-1TLC"
+			(at 236.22 100.33 0)
+			(hide yes)
+			(show_name no)
+			(do_not_autoplace no)
+			(effects
+				(font
+					(size 1.27 1.27)
+				)
+			)
+		)
+		(property "Datasheet" "https://www.coilcraft.com/getmedia/f685d903-2563-4c96-8ba6-f82a58883aeb/wbc.pdf"
+			(at 236.22 100.33 0)
+			(hide yes)
+			(show_name no)
+			(do_not_autoplace no)
+			(effects
+				(font
+					(size 1.27 1.27)
+				)
+			)
+		)
+		(property "Description" "1:2 impedance-ratio SMT wideband transformer, 0.2 MHz to 500 MHz, center-tapped secondary"
+			(at 236.22 100.33 0)
+			(hide yes)
+			(show_name no)
+			(do_not_autoplace no)
+			(effects
+				(font
+					(size 1.27 1.27)
+				)
+			)
+		)
+		(property "Manufacturer" "Coilcraft"
+			(at 236.22 100.33 0)
+			(hide yes)
+			(show_name no)
+			(do_not_autoplace no)
+			(effects
+				(font
+					(size 1.27 1.27)
+				)
+			)
+		)
+		(property "MPN" "WBC2-1TLC"
+			(at 236.22 100.33 0)
+			(hide yes)
+			(show_name no)
+			(do_not_autoplace no)
+			(effects
+				(font
+					(size 1.27 1.27)
+				)
+			)
+		)
+		(property "LCSC_PART" "C19191658"
+			(at 236.22 100.33 0)
+			(hide yes)
+			(show_name no)
+			(do_not_autoplace no)
+			(effects
+				(font
+					(size 1.27 1.27)
+				)
+			)
+		)
+		(pin "5"
+		)
+		(pin "4"
+		)
+		(pin "1"
+		)
+		(pin "3"
+		)
+		(pin "6"
+		)
+		(pin "2"
+		)
+		(instances
+			(project "WsprryPi Zero GPIO"
+				(path "/42fb2efa-c288-4686-a90a-043ad23a327d"
+					(reference "T41")
+					(unit 1)
+				)
