File: WsprryPi Zero GPIO/WsprryPi Zero GPIO.kicad_pcb (KiCad board)
At the start: 2 copper layers, 65 x 30 mm, 28 parts, among them J12 Conn_01x03, J41 SMA_Adafruit_1865, J42 J81/J82 LPF sockets, SW11 SKRPANE010, T21 WBC2-1TLC, T41 WBC2-1TLC, U11 Raspberry Pi 40-pin HAT inter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, U31 LTC6432AIUF-15#PBF, U51 TPS22918DBVR

Commit message: Address filled vias
Routing:
- net GND: track 38.9 -> 40.2 mm, vias 345 -> 387
