File: RPi Full-Size Hat Template/RPi Full-Size Hat Template.kicad_pcb (KiCad board)
At the start: 2 copper layers, 65 x 56.5 mm, 2 parts, among them U1 Raspberry Pi 40-pin HAT inter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

Commit message: Update HAT template references and localize Pico library assets
Parts:
- H1: footprint full-size-hat:Raspberry_Pi_HAT_2x20_Socket_3D -> full-size-hat-template:Raspberry_Pi_HAT_2x20_Socket_3D
- U1: footprint full-size-hat:Raspberry_Pi_HAT_Interface -> full-size-hat-template:Raspberry_Pi_HAT_Interface
Changed lines of the file:
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@@
 		)
 	)
-	(footprint "full-size-hat:Raspberry_Pi_HAT_Interface"
+	(footprint "full-size-hat-template:Raspberry_Pi_HAT_Interface"
 		(locked yes)
 		(layer "F.Cu")
@@
 		)
 		(sheetname "/")
-		(sheetfile "RPi Full-Size Hat.kicad_sch")
+		(sheetfile "RPi Full-Size Hat Template.kicad_sch")
 		(attr through_hole exclude_from_pos_files exclude_from_bom)
 		(duplicate_pad_numbers_are_jumpers no)
@@
 		(embedded_fonts no)
 	)
-	(footprint "full-size-hat:Raspberry_Pi_HAT_2x20_Socket_3D"
+	(footprint "full-size-hat-template:Raspberry_Pi_HAT_2x20_Socket_3D"
 		(layer "B.Cu")
 		(at 156.63 74.77 90)
@@
 		(duplicate_pad_numbers_are_jumpers no)
 		(embedded_fonts no)
-		(model "${KIPRJMOD}/full-size-hat.3dshapes/PinSocket_2x20_P2.54mm_Vertical.step"
+		(model "${KIPRJMOD}/full-size-hat-template.3dshapes/PinSocket_2x20_P2.54mm_Vertical.step"
 			(offset
 				(xyz 0 0 0)
