File: RPi Full-Size Hat Template/RPi Full-Size Hat Template.kicad_sch (KiCad schematic)
At the start: 2 parts, among them J1 Socket_2x20_P2.54mm, U1 Raspberry Pi 40-pin HAT inter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

Commit message: Update HAT template references and localize Pico library assets
Parts:
- J1: symbol full-size-hat:Socket_2x20_P2.54mm_BOM -> full-size-hat-template:Socket_2x20_P2.54mm_BOM
- U1: footprint full-size-hat:Raspberry_Pi_HAT_Interface -> full-size-hat-template:Raspberry_Pi_HAT_Interface; symbol full-size-hat:Raspberry_Pi_40_Pin_HAT_Interface -> full-size-hat-template:Raspberry_Pi_40_Pin_HAT_Interface
Changed lines of the file:
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@@
 	)
 	(symbol
-		(lib_id "full-size-hat:Socket_2x20_P2.54mm_BOM")
+		(lib_id "full-size-hat-template:Socket_2x20_P2.54mm_BOM")
 		(at 55.88 127 0)
 		(unit 1)
@@
 		)
 		(instances
-			(project "RPi Full-Size Hat"
+			(project "RPi Full-Size Hat Template"
 				(path "/42fb2efa-c288-4686-a90a-043ad23a327d"
 					(reference "J1")
@@
 	)
 	(symbol
-		(lib_id "full-size-hat:Raspberry_Pi_40_Pin_HAT_Interface")
+		(lib_id "full-size-hat-template:Raspberry_Pi_40_Pin_HAT_Interface")
 		(at 76.2 76.2 0)
 		(unit 1)
@@
 			)
 		)
-		(property "Footprint" "full-size-hat:Raspberry_Pi_HAT_Interface"
+		(property "Footprint" "full-size-hat-template:Raspberry_Pi_HAT_Interface"
 			(at 76.2 76.2 0)
 			(hide yes)
@@
 		)
 		(instances
-			(project "RPi Full-Size Hat"
+			(project "RPi Full-Size Hat Template"
 				(path "/42fb2efa-c288-4686-a90a-043ad23a327d"
 					(reference "U1")
