File: RPi Zero HAT Template/RPi Zero HAT Template.kicad_sch (KiCad schematic)
At the start: 2 parts, among them J1 Socket_2x20_P2.54mm, U1 Raspberry Pi 40-pin HAT inter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

Commit message: Update HAT template references and localize Pico library assets
Parts:
- J1: symbol zero-hat:Socket_2x20_P2.54mm_BOM -> zero-hat-template:Socket_2x20_P2.54mm_BOM
- U1: footprint zero-hat:Raspberry_Pi_Zero_HAT_Interface -> zero-hat-template:Raspberry_Pi_Zero_HAT_Interface; symbol zero-hat:Raspberry_Pi_40_Pin_HAT_Interface -> zero-hat-template:Raspberry_Pi_40_Pin_HAT_Interface
Changed lines of the file:
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@@
 	)
 	(symbol
-		(lib_id "zero-hat:Socket_2x20_P2.54mm_BOM")
+		(lib_id "zero-hat-template:Socket_2x20_P2.54mm_BOM")
 		(at 55.88 127 0)
 		(unit 1)
@@
 		)
 		(instances
-			(project "RPi Zero HAT"
+			(project "RPi Zero HAT Template"
 				(path "/42fb2efa-c288-4686-a90a-043ad23a327d"
 					(reference "J1")
@@
 	)
 	(symbol
-		(lib_id "zero-hat:Raspberry_Pi_40_Pin_HAT_Interface")
+		(lib_id "zero-hat-template:Raspberry_Pi_40_Pin_HAT_Interface")
 		(at 76.2 76.2 0)
 		(unit 1)
@@
 			)
 		)
-		(property "Footprint" "zero-hat:Raspberry_Pi_Zero_HAT_Interface"
+		(property "Footprint" "zero-hat-template:Raspberry_Pi_Zero_HAT_Interface"
 			(at 76.2 76.2 0)
 			(hide yes)
@@
 		)
 		(instances
-			(project "RPi Zero HAT"
+			(project "RPi Zero HAT Template"
 				(path "/42fb2efa-c288-4686-a90a-043ad23a327d"
 					(reference "U1")
