File: WsprryPi LPF/WsprryPi LPF.kicad_pcb (KiCad board)
At the start: 2 copper layers, 36.8 x 12.9 mm, 12 parts, among them J1 Jumper Pair

Commit message: Update LPF project names and references
Parts:
- CA1, CA3, CA5, CA7, CB1, CB3, CB5, CB7: footprint Wsprry Pi LPF:C_Disc_D3.0mm_W1.6mm_P2.50mm -> WsprryPi LPF:C_Disc_D3.0mm_W1.6mm_P2.50mm
- J1: footprint Wsprry Pi LPF:LPF_HeaderPair_2x1x04_P2.54mm_S33.02mm -> WsprryPi LPF:LPF_HeaderPair_2x1x04_P2.54mm_S33.02mm
- L2, L4, L6: footprint Wsprry Pi LPF:L_Axial_Horiz_Torroid_Vert_12mm_D5mm_P10.2mm -> WsprryPi LPF:L_Axial_Horiz_Torroid_Vert_12mm_D5mm_P10.2mm
Other:
- board text added: "WsprryPi LPF v1.0.1"
- board text removed: "Wsprry Pi LPF v1.0.1"
Changed lines of the file:
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@@
 	(paper "A")
 	(title_block
-		(title "Wsprry Pi LPF")
+		(title "WsprryPi LPF")
 		(date "2026-03-25")
 		(rev "1.0.2")
@@
 		)
 	)
-	(footprint "Wsprry Pi LPF:C_Disc_D3.0mm_W1.6mm_P2.50mm"
+	(footprint "WsprryPi LPF:C_Disc_D3.0mm_W1.6mm_P2.50mm"
 		(layer "F.Cu")
 		(at 150.49 95.34 -90)
@@
 		(property ki_fp_filters "C_*")
 		(sheetname "/")
-		(sheetfile "Wsprry-Pi-LPF.kicad_sch")
+		(sheetfile "WsprryPi LPF.kicad_sch")
 		(units
 			(unit
@@
 		)
 	)
-	(footprint "Wsprry Pi LPF:L_Axial_Horiz_Torroid_Vert_12mm_D5mm_P10.2mm"
+	(footprint "WsprryPi LPF:L_Axial_Horiz_Torroid_Vert_12mm_D5mm_P10.2mm"
 		(layer "F.Cu")
 		(at 146.125239 99.225 -90)
@@
 		(property ki_fp_filters "Inductor_* L_*")
 		(sheetname "/")
-		(sheetfile "Wsprry-Pi-LPF.kicad_sch")
+		(sheetfile "WsprryPi LPF.kicad_sch")
 		(units
 			(unit
@@
 		)
 	)
-	(footprint "Wsprry Pi LPF:L_Axial_Horiz_Torroid_Vert_12mm_D5mm_P10.2mm"
+	(footprint "WsprryPi LPF:L_Axial_Horiz_Torroid_Vert_12mm_D5mm_P10.2mm"
 		(layer "F.Cu")
 		(at 127.740477 99.225 -90)
@@
 		(property ki_fp_filters "Inductor_* L_*")
 		(sheetname "/")
-		(sheetfile "Wsprry-Pi-LPF.kicad_sch")
+		(sheetfile "WsprryPi LPF.kicad_sch")
 		(units
 			(unit
@@
 		)
 	)
-	(footprint "Wsprry Pi LPF:C_Disc_D3.0mm_W1.6mm_P2.50mm"
+	(footprint "WsprryPi LPF:C_Disc_D3.0mm_W1.6mm_P2.50mm"
 		(layer "F.Cu")
 		(at 133.182858 94.644664)
@@
 		(property ki_fp_filters "C_*")
 		(sheetname "/")
-		(sheetfile "Wsprry-Pi-LPF.kicad_sch")
+		(sheetfile "WsprryPi LPF.kicad_sch")
 		(units
 			(unit
@@
 		)
 	)
-	(footprint "Wsprry Pi LPF:C_Disc_D3.0mm_W1.6mm_P2.50mm"
+	(footprint "WsprryPi LPF:C_Disc_D3.0mm_W1.6mm_P2.50mm"
 		(layer "F.Cu")
 		(at 123.29 95.34 -90)
@@
 		(property ki_fp_filters "C_*")
 		(sheetname "/")
-		(sheetfile "Wsprry-Pi-LPF.kicad_sch")
+		(sheetfile "WsprryPi LPF.kicad_sch")
 		(units
 			(unit
@@
 		)
 	)
-	(footprint "Wsprry Pi LPF:L_Axial_Horiz_Torroid_Vert_12mm_D5mm_P10.2mm"
+	(footprint "WsprryPi LPF:L_Axial_Horiz_Torroid_Vert_12mm_D5mm_P10.2mm"
 		(layer "F.Cu")
 		(at 136.827858 99.074327 180)
@@
 		(property ki_fp_filters "Inductor_* L_*")
 		(sheetname "/")
-		(sheetfile "Wsprry-Pi-LPF.kicad_sch")
+		(sheetfile "WsprryPi LPF.kicad_sch")
 		(units
 			(unit
@@
 		)
 	)
-	(footprint "Wsprry Pi LPF:C_Disc_D3.0mm_W1.6mm_P2.50mm"
+	(footprint "WsprryPi LPF:C_Disc_D3.0mm_W1.6mm_P2.50mm"
 		(layer "F.Cu")
 		(at 123.29 102.84 90)
@@
 		(property ki_fp_filters "C_*")
 		(sheetname "/")
-		(sheetfile "Wsprry-Pi-LPF.kicad_sch")
+		(sheetfile "WsprryPi LPF.kicad_sch")
 		(units
 			(unit
@@
 		)
 	)
-	(footprint "Wsprry Pi LPF:C_Disc_D3.0mm_W1.6mm_P2.50mm"
+	(footprint "WsprryPi LPF:C_Disc_D3.0mm_W1.6mm_P2.50mm"
 		(layer "F.Cu")
 		(at 133.182858 103.539664)
@@
 		(property ki_fp_filters "C_*")
 		(sheetname "/")
-		(sheetfile "Wsprry-Pi-LPF.kicad_sch")
+		(sheetfile "WsprryPi LPF.kicad_sch")
 		(units
 			(unit
@@
 		)
 	)
-	(footprint "Wsprry Pi LPF:C_Disc_D3.0mm_W1.6mm_P2.50mm"
+	(footprint "WsprryPi LPF:C_Disc_D3.0mm_W1.6mm_P2.50mm"
 		(layer "F.Cu")
 		(at 140.682858 94.644664 180)
@@
 		(property ki_fp_filters "C_*")
 		(sheetname "/")
-		(sheetfile "Wsprry-Pi-LPF.kicad_sch")
+		(sheetfile "WsprryPi LPF.kicad_sch")
 		(units
 			(unit
@@
 		)
 	)
-	(footprint "Wsprry Pi LPF:C_Disc_D3.0mm_W1.6mm_P2.50mm"
+	(footprint "WsprryPi LPF:C_Disc_D3.0mm_W1.6mm_P2.50mm"
 		(layer "F.Cu")
 		(at 140.682858 103.539664 180)
@@
 		(property ki_fp_filters "C_*")
 		(sheetname "/")
-		(sheetfile "Wsprry-Pi-LPF.kicad_sch")
+		(sheetfile "WsprryPi LPF.kicad_sch")
 		(units
 			(unit
@@
 		)
 	)
-	(footprint "Wsprry Pi LPF:C_Disc_D3.0mm_W1.6mm_P2.50mm"
+	(footprint "WsprryPi LPF:C_Disc_D3.0mm_W1.6mm_P2.50mm"
 		(layer "F.Cu")
 		(at 150.49 102.84 90)
@@
 		(property ki_fp_filters "C_*")
 		(sheetname "/")
-		(sheetfile "Wsprry-Pi-LPF.kicad_sch")
+		(sheetfile "WsprryPi LPF.kicad_sch")
 		(units
 			(unit
@@
 		)
 	)
-	(footprint "Wsprry Pi LPF:LPF_HeaderPair_2x1x04_P2.54mm_S33.02mm"
+	(footprint "WsprryPi LPF:LPF_HeaderPair_2x1x04_P2.54mm_S33.02mm"
 		(layer "B.Cu")
 		(at 120.47 102.93)
-		(descr "Paired hand-fitted male 1x04 headers; 33.02 mm centerlines, 2.54 mm pitch; Wsprry LPF pinout, not QRP Labs electrical pinout")
+		(descr "Paired hand-fitted male 1x04 headers; 33.02 mm centerlines, 2.54 mm pitch; WsprryPi LPF pinout, not QRP Labs electrical pinout")
 		(tags "LPF paired header 33.02mm 1.300inch")
 		(property "Reference" "J1"
@@
 		)
 		(sheetname "/")
-		(sheetfile "Wsprry-Pi-LPF.kicad_sch")
+		(sheetfile "WsprryPi LPF.kicad_sch")
 		(units
 			(unit
@@
 		(layer "Edge.Cuts")
 	)
-	(gr_text "Wsprry Pi\nLPF v1.0.1"
+	(gr_text "WsprryPi\nLPF v1.0.1"
 		(at 136.98 99.01 0)
 		(layer "B.SilkS")

Commit message: File rename and cleanup
Parts:
- J1: value Jumper Pair -> LPF male headers; footprint WsprryPi LPF:LPF_HeaderPair_2x1x04_P2.54mm_S33.02mm -> WsprryPi LPF:LPF_HeaderPair_Male_2x1x04_P2.54mm_S33.02mm
Changed lines of the file:
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@@
 		)
 	)
-	(footprint "WsprryPi LPF:LPF_HeaderPair_2x1x04_P2.54mm_S33.02mm"
+	(footprint "WsprryPi LPF:LPF_HeaderPair_Male_2x1x04_P2.54mm_S33.02mm"
 		(layer "B.Cu")
 		(at 120.47 102.93)
@@
 			)
 		)
-		(property "Value" "Jumper Pair"
+		(property "Value" "LPF male headers"
 			(at 16.51 -11 180)
 			(layer "B.Fab")

Commit message: Prep for assembly
Other:
- board text added: "WsprryPi LPF v1.0.0"
- board text removed: "WsprryPi LPF v1.0.1"
Changed lines of the file:
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@@
 	(title_block
 		(title "WsprryPi LPF")
-		(date "2026-03-25")
-		(rev "1.0.2")
+		(date "2026-10-05")
+		(rev "1.0.0")
 	)
 	(layers
@@
 		(layer "Edge.Cuts")
 	)
-	(gr_text "WsprryPi\nLPF v1.0.1"
+	(gr_text "WsprryPi\nLPF v1.0.0"
 		(at 136.98 99.01 0)
 		(layer "B.SilkS")
