File: WsprryPi LPF/WsprryPi LPF.kicad_sch (KiCad schematic)
At the start: 12 parts, among them J1 Jumper Pair

Commit message: Update LPF project names and references
Parts:
- CA1, CA3, CA5, CA7, CB1, CB3, CB5, CB7: footprint Wsprry Pi LPF:C_Disc_D3.0mm_W1.6mm_P2.50mm -> WsprryPi LPF:C_Disc_D3.0mm_W1.6mm_P2.50mm; symbol Wsprry Pi LPF:C -> WsprryPi LPF:C
- J1: footprint Wsprry Pi LPF:LPF_HeaderPair_2x1x04_P2.54mm_S33.02mm -> WsprryPi LPF:LPF_HeaderPair_2x1x04_P2.54mm_S33.02mm; symbol Wsprry Pi LPF:LPF_HeaderPair_2x1x04_P2.54mm_S33.02mm -> WsprryPi LPF:LPF_HeaderPair_2x1x04_P2.54mm_S33.02mm
- L2, L4, L6: footprint Wsprry Pi LPF:L_Axial_Horiz_Torroid_Vert_12mm_D5mm_P10.2mm -> WsprryPi LPF:L_Axial_Horiz_Torroid_Vert_12mm_D5mm_P10.2mm; symbol Wsprry Pi LPF:L -> WsprryPi LPF:L
Other:
- title: Wsprry Pi LPF -> WsprryPi LPF
Changed lines of the file:
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@@
 	(paper "A")
 	(title_block
-		(title "Wsprry Pi LPF")
+		(title "WsprryPi LPF")
 		(date "2026-03-26")
 		(rev "1.0.2")
@@
 	)
 	(symbol
-		(lib_id "Wsprry Pi LPF:LPF_HeaderPair_2x1x04_P2.54mm_S33.02mm")
+		(lib_id "WsprryPi LPF:LPF_HeaderPair_2x1x04_P2.54mm_S33.02mm")
 		(at 137.16 124.46 0)
 		(unit 1)
@@
 			)
 		)
-		(property "Footprint" "Wsprry Pi LPF:LPF_HeaderPair_2x1x04_P2.54mm_S33.02mm"
+		(property "Footprint" "WsprryPi LPF:LPF_HeaderPair_2x1x04_P2.54mm_S33.02mm"
 			(at 137.16 124.46 0)
 			(hide yes)
@@
 		)
 		(instances
-			(project "Wsprry-Pi-LPF"
+			(project "WsprryPi LPF"
 				(path "/a5c3480f-f07b-4318-b0ac-3cbcb5b2943e"
 					(reference "J1")
@@
 	)
 	(symbol
-		(lib_id "Wsprry Pi LPF:GND")
+		(lib_id "WsprryPi LPF:GND")
 		(at 152.4 118.11 180)
 		(unit 1)
@@
 		)
 		(instances
-			(project "Wsprry-Pi-LPF"
+			(project "WsprryPi LPF"
 				(path "/a5c3480f-f07b-4318-b0ac-3cbcb5b2943e"
 					(reference "#PWR025")
@@
 	)
 	(symbol
-		(lib_id "Wsprry Pi LPF:C")
+		(lib_id "WsprryPi LPF:C")
 		(at 101.6 92.71 0)
 		(unit 1)
@@
 			)
 		)
-		(property "Footprint" "Wsprry Pi LPF:C_Disc_D3.0mm_W1.6mm_P2.50mm"
+		(property "Footprint" "WsprryPi LPF:C_Disc_D3.0mm_W1.6mm_P2.50mm"
 			(at 102.5652 96.52 0)
 			(hide yes)
@@
 		)
 		(instances
-			(project "Wsprry-Pi-LPF"
+			(project "WsprryPi LPF"
 				(path "/a5c3480f-f07b-4318-b0ac-3cbcb5b2943e"
 					(reference "CA1")
@@
 	)
 	(symbol
-		(lib_id "Wsprry Pi LPF:C")
+		(lib_id "WsprryPi LPF:C")
 		(at 142.24 92.71 0)
 		(unit 1)
@@
 			)
 		)
-		(property "Footprint" "Wsprry Pi LPF:C_Disc_D3.0mm_W1.6mm_P2.50mm"
+		(property "Footprint" "WsprryPi LPF:C_Disc_D3.0mm_W1.6mm_P2.50mm"
 			(at 143.2052 96.52 0)
 			(hide yes)
@@
 		)
 		(instances
-			(project "Wsprry-Pi-LPF"
+			(project "WsprryPi LPF"
 				(path "/a5c3480f-f07b-4318-b0ac-3cbcb5b2943e"
 					(reference "CA5")
@@
 	)
 	(symbol
-		(lib_id "Wsprry Pi LPF:C")
+		(lib_id "WsprryPi LPF:C")
 		(at 172.72 92.71 0)
 		(unit 1)
@@
 			)
 		)
-		(property "Footprint" "Wsprry Pi LPF:C_Disc_D3.0mm_W1.6mm_P2.50mm"
+		(property "Footprint" "WsprryPi LPF:C_Disc_D3.0mm_W1.6mm_P2.50mm"
 			(at 173.6852 96.52 0)
 			(hide yes)
@@
 		)
 		(instances
-			(project "Wsprry-Pi-LPF"
+			(project "WsprryPi LPF"
 				(path "/a5c3480f-f07b-4318-b0ac-3cbcb5b2943e"
 					(reference "CB7")
@@
 	)
 	(symbol
-		(lib_id "Wsprry Pi LPF:L")
+		(lib_id "WsprryPi LPF:L")
 		(at 116.84 105.41 180)
 		(unit 1)
@@
 			)
 		)
-		(property "Footprint" "Wsprry Pi LPF:L_Axial_Horiz_Torroid_Vert_12mm_D5mm_P10.2mm"
+		(property "Footprint" "WsprryPi LPF:L_Axial_Horiz_Torroid_Vert_12mm_D5mm_P10.2mm"
 			(at 116.84 105.41 0)
 			(hide yes)
@@
 		)
 		(instances
-			(project "Wsprry-Pi-LPF"
+			(project "WsprryPi LPF"
 				(path "/a5c3480f-f07b-4318-b0ac-3cbcb5b2943e"
 					(reference "L2")
@@
 	)
 	(symbol
-		(lib_id "Wsprry Pi LPF:C")
+		(lib_id "WsprryPi LPF:C")
 		(at 121.92 92.71 0)
 		(unit 1)
@@
 			)
 		)
-		(property "Footprint" "Wsprry Pi LPF:C_Disc_D3.0mm_W1.6mm_P2.50mm"
+		(property "Footprint" "WsprryPi LPF:C_Disc_D3.0mm_W1.6mm_P2.50mm"
 			(at 122.8852 96.52 0)
 			(hide yes)
@@
 		)
 		(instances
-			(project "Wsprry-Pi-LPF"
+			(project "WsprryPi LPF"
 				(path "/a5c3480f-f07b-4318-b0ac-3cbcb5b2943e"
 					(reference "CA3")
@@
 	)
 	(symbol
-		(lib_id "Wsprry Pi LPF:L")
+		(lib_id "WsprryPi LPF:L")
 		(at 157.48 105.41 180)
 		(unit 1)
@@
 			)
 		)
-		(property "Footprint" "Wsprry Pi LPF:L_Axial_Horiz_Torroid_Vert_12mm_D5mm_P10.2mm"
+		(property "Footprint" "WsprryPi LPF:L_Axial_Horiz_Torroid_Vert_12mm_D5mm_P10.2mm"
 			(at 157.48 105.41 0)
 			(hide yes)
@@
 		)
 		(instances
-			(project "Wsprry-Pi-LPF"
+			(project "WsprryPi LPF"
 				(path "/a5c3480f-f07b-4318-b0ac-3cbcb5b2943e"
 					(reference "L6")
@@
 	)
 	(symbol
-		(lib_id "Wsprry Pi LPF:GND")
+		(lib_id "WsprryPi LPF:GND")
 		(at 167.64 86.36 180)
 		(unit 1)
@@
 		)
 		(instances
-			(project "Wsprry-Pi-LPF"
+			(project "WsprryPi LPF"
 				(path "/a5c3480f-f07b-4318-b0ac-3cbcb5b2943e"
 					(reference "#PWR01")
@@
 	)
 	(symbol
-		(lib_id "Wsprry Pi LPF:C")
+		(lib_id "WsprryPi LPF:C")
 		(at 132.08 92.71 0)
 		(unit 1)
@@
 			)
 		)
-		(property "Footprint" "Wsprry Pi LPF:C_Disc_D3.0mm_W1.6mm_P2.50mm"
+		(property "Footprint" "WsprryPi LPF:C_Disc_D3.0mm_W1.6mm_P2.50mm"
 			(at 133.0452 96.52 0)
 			(hide yes)
@@
 		)
 		(instances
-			(project "Wsprry-Pi-LPF"
+			(project "WsprryPi LPF"
 				(path "/a5c3480f-f07b-4318-b0ac-3cbcb5b2943e"
 					(reference "CB3")
@@
 	)
 	(symbol
-		(lib_id "Wsprry Pi LPF:C")
+		(lib_id "WsprryPi LPF:C")
 		(at 111.76 92.71 0)
 		(unit 1)
@@
 			)
 		)
-		(property "Footprint" "Wsprry Pi LPF:C_Disc_D3.0mm_W1.6mm_P2.50mm"
+		(property "Footprint" "WsprryPi LPF:C_Disc_D3.0mm_W1.6mm_P2.50mm"
 			(at 112.7252 96.52 0)
 			(hide yes)
@@
 		)
 		(instances
-			(project "Wsprry-Pi-LPF"
+			(project "WsprryPi LPF"
 				(path "/a5c3480f-f07b-4318-b0ac-3cbcb5b2943e"
 					(reference "CB1")
@@
 	)
 	(symbol
-		(lib_id "Wsprry Pi LPF:GND")
+		(lib_id "WsprryPi LPF:GND")
 		(at 106.68 86.36 180)
 		(unit 1)
@@
 		)
 		(instances
-			(project "Wsprry-Pi-LPF"
+			(project "WsprryPi LPF"
 				(path "/a5c3480f-f07b-4318-b0ac-3cbcb5b2943e"
 					(reference "#PWR04")
@@
 	)
 	(symbol
-		(lib_id "Wsprry Pi LPF:GND")
+		(lib_id "WsprryPi LPF:GND")
 		(at 121.92 128.27 0)
 		(unit 1)
@@
 		)
 		(instances
-			(project "Wsprry-Pi-LPF"
+			(project "WsprryPi LPF"
 				(path "/a5c3480f-f07b-4318-b0ac-3cbcb5b2943e"
 					(reference "#PWR021")
@@
 	)
 	(symbol
-		(lib_id "Wsprry Pi LPF:GND")
+		(lib_id "WsprryPi LPF:GND")
 		(at 152.4 128.27 0)
 		(unit 1)
@@
 		)
 		(instances
-			(project "Wsprry-Pi-LPF"
+			(project "WsprryPi LPF"
 				(path "/a5c3480f-f07b-4318-b0ac-3cbcb5b2943e"
 					(reference "#PWR020")
@@
 	)
 	(symbol
-		(lib_id "Wsprry Pi LPF:GND")
+		(lib_id "WsprryPi LPF:GND")
 		(at 121.92 118.11 180)
 		(unit 1)
@@
 		)
 		(instances
-			(project "Wsprry-Pi-LPF"
+			(project "WsprryPi LPF"
 				(path "/a5c3480f-f07b-4318-b0ac-3cbcb5b2943e"
 					(reference "#PWR024")
@@
 	)
 	(symbol
-		(lib_id "Wsprry Pi LPF:GND")
+		(lib_id "WsprryPi LPF:GND")
 		(at 147.32 86.36 180)
 		(unit 1)
@@
 		)
 		(instances
-			(project "Wsprry-Pi-LPF"
+			(project "WsprryPi LPF"
 				(path "/a5c3480f-f07b-4318-b0ac-3cbcb5b2943e"
 					(reference "#PWR03")
@@
 	)
 	(symbol
-		(lib_id "Wsprry Pi LPF:C")
+		(lib_id "WsprryPi LPF:C")
 		(at 162.56 92.71 0)
 		(unit 1)
@@
 			)
 		)
-		(property "Footprint" "Wsprry Pi LPF:C_Disc_D3.0mm_W1.6mm_P2.50mm"
+		(property "Footprint" "WsprryPi LPF:C_Disc_D3.0mm_W1.6mm_P2.50mm"
 			(at 163.5252 96.52 0)
 			(hide yes)
@@
 		)
 		(instances
-			(project "Wsprry-Pi-LPF"
+			(project "WsprryPi LPF"
 				(path "/a5c3480f-f07b-4318-b0ac-3cbcb5b2943e"
 					(reference "CA7")
@@
 	)
 	(symbol
-		(lib_id "Wsprry Pi LPF:GND")
+		(lib_id "WsprryPi LPF:GND")
 		(at 127 86.36 180)
 		(unit 1)
@@
 		)
 		(instances
-			(project "Wsprry-Pi-LPF"
+			(project "WsprryPi LPF"
 				(path "/a5c3480f-f07b-4318-b0ac-3cbcb5b2943e"
 					(reference "#PWR02")
@@
 	)
 	(symbol
-		(lib_id "Wsprry Pi LPF:PWR_FLAG")
+		(lib_id "WsprryPi LPF:PWR_FLAG")
 		(at 118.11 119.38 0)
 		(unit 1)
@@
 		)
 		(instances
-			(project "Wsprry-Pi-LPF"
+			(project "WsprryPi LPF"
 				(path "/a5c3480f-f07b-4318-b0ac-3cbcb5b2943e"
 					(reference "#FLG01")
@@
 	)
 	(symbol
-		(lib_id "Wsprry Pi LPF:L")
+		(lib_id "WsprryPi LPF:L")
 		(at 137.16 105.41 180)
 		(unit 1)
@@
 			)
 		)
-		(property "Footprint" "Wsprry Pi LPF:L_Axial_Horiz_Torroid_Vert_12mm_D5mm_P10.2mm"
+		(property "Footprint" "WsprryPi LPF:L_Axial_Horiz_Torroid_Vert_12mm_D5mm_P10.2mm"
 			(at 137.16 105.41 0)
 			(hide yes)
@@
 		)
 		(instances
-			(project "Wsprry-Pi-LPF"
+			(project "WsprryPi LPF"
 				(path "/a5c3480f-f07b-4318-b0ac-3cbcb5b2943e"
 					(reference "L4")
@@
 	)
 	(symbol
-		(lib_id "Wsprry Pi LPF:C")
+		(lib_id "WsprryPi LPF:C")
 		(at 152.4 92.71 0)
 		(unit 1)
@@
 			)
 		)
-		(property "Footprint" "Wsprry Pi LPF:C_Disc_D3.0mm_W1.6mm_P2.50mm"
+		(property "Footprint" "WsprryPi LPF:C_Disc_D3.0mm_W1.6mm_P2.50mm"
 			(at 153.3652 96.52 0)
 			(hide yes)
@@
 		)
 		(instances
-			(project "Wsprry-Pi-LPF"
+			(project "WsprryPi LPF"
 				(path "/a5c3480f-f07b-4318-b0ac-3cbcb5b2943e"
 					(reference "CB5")

Commit message: File rename and cleanup
Parts:
- J1: value Jumper Pair -> LPF male headers; footprint WsprryPi LPF:LPF_HeaderPair_2x1x04_P2.54mm_S33.02mm -> WsprryPi LPF:LPF_HeaderPair_Male_2x1x04_P2.54mm_S33.02mm; symbol WsprryPi LPF:LPF_HeaderPair_2x1x04_P2.54mm_S33.02mm -> WsprryPi LPF:LPF_HeaderPair_Male_2x1x04_P2.54mm_S33.02mm
Changed lines of the file:
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@@
 	)
 	(symbol
-		(lib_id "WsprryPi LPF:LPF_HeaderPair_2x1x04_P2.54mm_S33.02mm")
+		(lib_id "WsprryPi LPF:LPF_HeaderPair_Male_2x1x04_P2.54mm_S33.02mm")
 		(at 137.16 124.46 0)
 		(unit 1)
@@
 			)
 		)
-		(property "Value" "Jumper Pair"
+		(property "Value" "LPF male headers"
 			(at 137.16 114.3 0)
 			(show_name no)
@@
 			)
 		)
-		(property "Footprint" "WsprryPi LPF:LPF_HeaderPair_2x1x04_P2.54mm_S33.02mm"
+		(property "Footprint" "WsprryPi LPF:LPF_HeaderPair_Male_2x1x04_P2.54mm_S33.02mm"
 			(at 137.16 124.46 0)
 			(hide yes)
