File: WsprryPi Zero GPIO BS170/WsprryPi Zero GPIO BS170.kicad_pcb (KiCad board)
At the start: 2 copper layers, 65 x 30 mm, 26 parts, among them J12 GPIO, J21 BIAS_SET, J51 SMA_Adafruit_1865, J52 LPF female headers, Q41 BS170, SW11 SKRPANE010, U11 Raspberry Pi 40-pin HAT inter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, U21 TPS22918DBVR

Commit message: Prep for assembly
Parts:
- C31, C51: footprint wsprrypi-zero-gpio-bs170:C_0603_1608Metric -> wsprrypi-zero-gpio-bs170:C_1206_3216Metric
- moved C31 6.70 mm to (107.7, 90.5), turned to -90 degrees
- moved RV31 2.80 mm to (104.7, 90.4)
- moved C51 0.90 mm to (119.7, 96.8)
- moved C32 0.84 mm to (107.8, 98.7)
- moved Q41 0.84 mm to (115.8, 96.0)
- moved R31 0.84 mm to (111.6, 96.4)
- moved R33 0.84 mm to (113.1, 96.4)
- moved R32 0.84 mm to (110.8, 98.7)
- moved L41 0.50 mm to (115.1, 88.0)
Connections:
- C41 pad 1: /BIAS -> /SW_5V
- C42 pad 1: /BIAS -> /SW_5V
- L41 pad 1: /BIAS -> /SW_5V
- R41 pad 2: /BIAS -> /SW_5V
- RV31 pad 1: /BIAS -> /SW_5V
Routing:
- net /BIAS: track 12.8 -> 0.00 mm
- net /SW_5V: track 19.6 -> 31.8 mm
- net /GPIO_RF: track 34.2 -> 27.4 mm
- net Net-(C31-Pad2): track 1.46 -> 6.15 mm
- net /PA_DRAIN: track 11.2 -> 7.09 mm
- net GND: track 28.9 -> 32.0 mm, vias 171 -> 296
- net Net-(C32-Pad2): track 7.56 -> 9.78 mm
- net /FINAL_OUT: track 5.38 -> 6.42 mm
- net /GPIO20: track 30.9 -> 31.8 mm
