File: WsprryPi Zero GPIO BS170/WsprryPi Zero GPIO BS170.kicad_sch (KiCad schematic)
At the start: 26 parts, among them J11 Socket_2x20_P2.54mm, J12 Conn_01x03, J51 SMA_Adafruit_1865, J52 LPF female headers, Q41 BS170, SW11 SKRPANE010, U11 Raspberry Pi 40-pin HAT inter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, U21 TPS22918DBVR

Commit message: Add bias set
Parts:
- added J21: Conn_01x02, wsprrypi-zero-gpio-bs170:PinHeader_1x02_P2.54mm_Vertical, symbol wsprrypi-zero-gpio-bs170:Conn_01x02
Connections:
- net GND: now also C21.2, C41.2, C42.2; no longer C21.1, C41.1, C42.1
- net PI_5V: now also C21.1, J21.1 (Pin_1); no longer C21.2
- net SW_5V: now also R22.1, J21.2 (Pin_2); no longer R22.2
- net at U21.5 (QOD): now also R22.2; no longer R22.1
- net PRE_CHOKE renamed BIAS
- net BIAS: now also C41.1, C42.1; no longer C41.2, C42.2
Other:
- note added: "BIAS SET - normally open"
- moved on the sheet: C21, C41, C42, R22
Changed lines of the file:
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@@
 	)
 	(junction
-		(at 107.95 92.71)
+		(at 161.29 31.75)
 		(diameter 0)
 		(color 0 0 0 0)
 	)
 	(junction
-		(at 161.29 31.75)
+		(at 107.95 92.71)
 		(diameter 0)
 		(color 0 0 0 0)
@@
 	(wire
 		(pts
-			(xy 161.29 31.75) (xy 161.29 33.02)
-		)
-		(stroke
-			(width 0)
-			(type default)
-		)
-	)
-	(wire
-		(pts
 			(xy 106.68 92.71) (xy 107.95 92.71)
 		)
@@
 	(wire
 		(pts
-			(xy 95.25 50.8) (xy 106.68 50.8)
-		)
-		(stroke
-			(width 0)
-			(type default)
-		)
-	)
-	(wire
-		(pts
 			(xy 162.56 22.86) (xy 161.29 22.86)
 		)
@@
 	(wire
 		(pts
+			(xy 156.21 31.75) (xy 161.29 31.75)
+		)
+		(stroke
+			(width 0)
+			(type default)
+		)
+	)
+	(wire
+		(pts
 			(xy 110.49 46.99) (xy 110.49 45.72)
 		)
@@
 	(wire
 		(pts
+			(xy 161.29 31.75) (xy 161.29 33.02)
+		)
+		(stroke
+			(width 0)
+			(type default)
+		)
+	)
+	(wire
+		(pts
 			(xy 120.65 45.72) (xy 121.92 45.72)
 		)
@@
 	(wire
 		(pts
-			(xy 240.03 80.01) (xy 240.03 81.28)
+			(xy 106.68 50.8) (xy 101.6 50.8)
 		)
 		(stroke
@@
 	(wire
 		(pts
-			(xy 99.06 82.55) (xy 97.79 82.55)
+			(xy 240.03 80.01) (xy 240.03 81.28)
 		)
 		(stroke
@@
 	(wire
 		(pts
-			(xy 161.29 22.86) (xy 161.29 29.21)
+			(xy 99.06 82.55) (xy 97.79 82.55)
 		)
 		(stroke
@@
 	(wire
 		(pts
-			(xy 149.86 31.75) (xy 161.29 31.75)
+			(xy 161.29 22.86) (xy 161.29 29.21)
 		)
 		(stroke
@@
 		)
 	)
-	(label "PRE_CHOKE"
-		(at 149.86 31.75 0)
-		(effects
-			(font
-				(size 1.27 1.27)
-			)
-			(justify left bottom)
-		)
-	)
-	(label "PRE_CHOKE"
-		(at 95.25 50.8 0)
+	(label "BIAS"
+		(at 156.21 31.75 0)
 		(effects
 			(font
@@
 		)
 	)
+	(label "BIAS"
+		(at 101.6 50.8 0)
+		(effects
+			(font
+				(size 1.27 1.27)
+			)
+			(justify left bottom)
+		)
+	)
 	(label "AMP_EN"
 		(at 17.78 69.85 0)
@@
 	(symbol
 		(lib_id "wsprrypi-zero-gpio-bs170:C_0603")
-		(at 166.37 29.21 180)
+		(at 166.37 29.21 0)
 		(unit 1)
 		(body_style 1)
@@
 		(dnp no)
 		(property "Reference" "C41"
-			(at 168.91 27.432 0)
+			(at 163.83 27.94 0)
 			(show_name no)
 			(do_not_autoplace no)
@@
 		)
 		(property "Value" "100nF"
-			(at 170.18 30.734 0)
+			(at 170.18 30.48 0)
 			(show_name no)
 			(do_not_autoplace no)
@@
 	(symbol
 		(lib_id "wsprrypi-zero-gpio-bs170:C_0805")
-		(at 166.37 22.86 180)
+		(at 166.37 22.86 0)
 		(unit 1)
 		(body_style 1)
@@
 		(dnp no)
 		(property "Reference" "C42"
-			(at 168.91 21.336 0)
+			(at 163.83 24.384 0)
 			(show_name no)
 			(do_not_autoplace no)
@@
 		)
 		(property "Value" "1µF"
-			(at 169.164 24.13 0)
+			(at 169.164 21.59 0)
 			(show_name no)
 			(do_not_autoplace no)
@@
 	(symbol
 		(lib_id "wsprrypi-zero-gpio-bs170:C_0805")
-		(at 102.87 82.55 0)
+		(at 102.87 82.55 180)
 		(unit 1)
 		(body_style 1)
@@
 		(dnp no)
 		(property "Reference" "C21"
-			(at 102.87 78.232 0)
+			(at 102.87 80.264 0)
 			(show_name no)
 			(do_not_autoplace no)
@@
 		)
 		(property "Value" "10µF"
-			(at 102.87 80.01 0)
+			(at 102.87 85.09 0)
 			(show_name no)
 			(do_not_autoplace no)
@@
 	(symbol
 		(lib_id "wsprrypi-zero-gpio-bs170:R_0603")
-		(at 138.43 86.36 0)
+		(at 138.43 86.36 180)
 		(unit 1)
 		(body_style 1)
@@
 		)
 		(property "Footprint" "wsprrypi-zero-gpio-bs170:R_0603_1608Metric"
-			(at 139.13 86.65 0)
+			(at 137.73 86.07 0)
 			(hide yes)
 			(show_name no)
@@
 		)
 		(property "Datasheet" "~"
-			(at 139.13 86.65 0)
+			(at 137.73 86.07 0)
 			(hide yes)
 			(show_name no)
@@
 		)
 		(property "Description" "Generic resistor using a compact US zigzag symbol and the local KiCad 0603 metric footprint"
-			(at 139.13 86.65 0)
+			(at 137.73 86.07 0)
 			(hide yes)
 			(show_name no)
@@
 	)
 	(embedded_fonts no)
+	(wire
+		(pts
+			(xy 138.43 96.52) (xy 146.05 96.52)
+		)
+		(stroke
+			(width 0)
+			(type default)
+		)
+	)
+	(label "PI_5V"
+		(at 138.43 96.52 0)
+		(effects
+			(font
+				(size 1.27 1.27)
+			)
+			(justify left bottom)
+		)
+	)
+	(wire
+		(pts
+			(xy 138.43 99.06) (xy 146.05 99.06)
+		)
+		(stroke
+			(width 0)
+			(type default)
+		)
+	)
+	(label "SW_5V"
+		(at 138.43 99.06 0)
+		(effects
+			(font
+				(size 1.27 1.27)
+			)
+			(justify left bottom)
+		)
+	)
+	(text "BIAS SET - normally open"
+		(exclude_from_sim no)
+		(at 135.89 103.505 0)
+		(effects
+			(font
+				(size 1.016 1.016)
+			)
+			(justify left bottom)
+		)
+	)
+	(symbol
+		(lib_id "wsprrypi-zero-gpio-bs170:Conn_01x02")
+		(at 151.13 96.52 0)
+		(unit 1)
+		(body_style 1)
+		(exclude_from_sim no)
+		(in_bom no)
+		(on_board yes)
+		(in_pos_files no)
+		(dnp no)
+		(property "Reference" "J21"
+			(at 151.13 93.98 0)
+			(show_name no)
+			(do_not_autoplace no)
+			(effects
+				(font
+					(size 1.27 1.27)
+				)
+			)
+		)
+		(property "Value" "Conn_01x02"
+			(at 151.13 101.6 0)
+			(hide yes)
+			(show_name no)
+			(do_not_autoplace no)
+			(effects
+				(font
+					(size 1.27 1.27)
+				)
+			)
+		)
+		(property "Footprint" "wsprrypi-zero-gpio-bs170:PinHeader_1x02_P2.54mm_Vertical"
+			(at 151.13 96.52 0)
+			(hide yes)
+			(show_name no)
+			(do_not_autoplace no)
+			(effects
+				(font
+					(size 1.27 1.27)
+				)
+			)
+		)
+		(property "Datasheet" ""
+			(at 151.13 96.52 0)
+			(hide yes)
+			(show_name no)
+			(do_not_autoplace no)
+			(effects
+				(font
+					(size 1.27 1.27)
+				)
+			)
+		)
+		(property "Description" "Normally open bias-setting supply bypass; pin 1 PI_5V, pin 2 SW_5V; same 2.54 mm male header style as J12"
+			(at 151.13 96.52 0)
+			(hide yes)
+			(show_name no)
+			(do_not_autoplace no)
+			(effects
+				(font
+					(size 1.27 1.27)
+				)
+			)
+		)
+		(pin "1"
+		)
+		(pin "2"
+		)
+		(instances
+			(project "WsprryPi Zero GPIO BS170"
+				(path "/42fb2efa-c288-4686-a90a-043ad23a327d"
+					(reference "J21")
+					(unit 1)
+				)
+			)
+		)
+	)
 )

Commit message: Update with part selections
Parts:
- C21: LCSC_PART C15850 -> C20070397; MPN (none) -> CSA0805X5R106K250MT; Manufacturer (none) -> HRE
- C22: MPN (none) -> CL10B102KB8NNNC; Manufacturer (none) -> Samsung Electro-Mechanics
- C23: LCSC_PART C28323 -> C726584; MPN (none) -> AC0805KKX7R9BB105; Manufacturer (none) -> YAGEO
- C31, C32, C41, C51: LCSC_PART (none) -> C235731; MPN (none) -> FN18X104K500PBG; Manufacturer (none) -> PSA
- C42: LCSC_PART (none) -> C726584; MPN (none) -> AC0805KKX7R9BB105; Manufacturer (none) -> YAGEO
- D11: value KT-0603W -> KT-0603R; MPN (none) -> KT-0603R; Manufacturer (none) -> Hubei KENTO Elec
- J12: value Conn_01x03 -> GPIO
- J21: value Conn_01x02 -> BIAS_SET
- Q41: now left out of the parts list
- R11: LCSC_PART C22962 -> C2907014; MPN (none) -> FRC0603F2200TS; Manufacturer (none) -> FOJAN
- R21: LCSC_PART C14675 -> C25803; MPN (none) -> 0603WAF1003T5E; Manufacturer (none) -> UNI-ROYAL
- R22: MPN (none) -> FRC0603F1001TS; Manufacturer (none) -> FOJAN
- R31: LCSC_PART (none) -> C23345; MPN (none) -> 0603WAF220JT5E; Manufacturer (none) -> UNI-ROYAL
- R32: LCSC_PART (none) -> C23162; MPN (none) -> 0603WAF4701T5E; Manufacturer (none) -> UNI-ROYAL
- R33: LCSC_PART (none) -> C25803; MPN (none) -> 0603WAF1003T5E; Manufacturer (none) -> UNI-ROYAL
- R41: LCSC_PART (none) -> C2907288; MPN (none) -> FRC0805P000 TS; Manufacturer (none) -> FOJAN
- RV31: Manufacturer Bourns -> BOURNS
- SW11: Manufacturer Alps Alpine -> ALPSALPINE
- U21: Manufacturer Texas Instruments -> TI

Commit message: Prep for assembly
Parts:
- C21: LCSC Part # (none) -> C20070397; LCSC_PART C20070397 -> (none)
- C22: LCSC Part # (none) -> C1588; LCSC_PART C1588 -> (none)
- C23, C42: LCSC Part # (none) -> C726584; LCSC_PART C726584 -> (none)
- C31, C51: footprint wsprrypi-zero-gpio-bs170:C_0603_1608Metric -> wsprrypi-zero-gpio-bs170:C_1206_3216Metric; LCSC Part # (none) -> C170182; LCSC_PART C235731 -> (none); MPN FN18X104K500PBG -> 1206N104J500CT; Manufacturer PSA -> Walsin
- C32, C41: LCSC Part # (none) -> C235731; LCSC_PART C235731 -> (none)
- D11: LCSC Part # (none) -> C2286; LCSC_PART C2286 -> (none)
- R11: LCSC Part # (none) -> C2907014; LCSC_PART C2907014 -> (none)
- R21, R33: LCSC Part # (none) -> C25803; LCSC_PART C25803 -> (none)
- R22: LCSC Part # (none) -> C2907002; LCSC_PART C2907002 -> (none)
- R31: LCSC Part # (none) -> C23345; LCSC_PART C23345 -> (none)
- R32: LCSC Part # (none) -> C23162; LCSC_PART C23162 -> (none)
- R41: symbol wsprrypi-zero-gpio-bs170:R_0805 -> wsprrypi-zero-gpio-bs170:R_0805_0R_Jumper; LCSC Part # (none) -> C2907288; LCSC_PART C2907288 -> (none)
- RV31: LCSC Part # (none) -> C719177; LCSC_PART C719177 -> (none)
- SW11: LCSC Part # (none) -> C470426; LCSC_PART C470426 -> (none)
- U21: LCSC Part # (none) -> C131941; LCSC_PART C131941 -> (none)
Connections:
- net BIAS is gone; now on net SW_5V: C41.1, C42.1, L41.1, R41.2, RV31.1
Changed lines of the file:
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@@
 		)
 	)
-	(label "BIAS"
+	(label "SW_5V"
 		(at 156.21 31.75 0)
 		(effects
@@
 		)
 	)
-	(label "BIAS"
+	(label "SW_5V"
 		(at 101.6 50.8 0)
 		(effects
@@
 			)
 		)
-		(property "LCSC_PART" "C235731"
+		(property "LCSC Part #" "C235731"
 			(at 166.37 29.21 0)
 			(hide yes)
@@
 			)
 		)
-		(property "LCSC_PART" "C23345"
+		(property "LCSC Part #" "C23345"
 			(at 115.57 26.67 0)
 			(hide yes)
@@
 			)
 		)
-		(property "LCSC_PART" "C235731"
+		(property "LCSC Part #" "C235731"
 			(at 120.65 50.8 0)
 			(hide yes)
@@
 		(lib_id "wsprrypi-zero-gpio-bs170:C_0603")
 		(at 106.68 26.67 0)
+		(mirror x)
 		(unit 1)
 		(body_style 1)
@@
 		(dnp no)
 		(property "Reference" "C31"
-			(at 106.68 21.59 0)
+			(at 106.68 24.13 0)
 			(show_name no)
 			(do_not_autoplace no)
@@
 		)
 		(property "Value" "100nF"
-			(at 106.68 24.13 0)
+			(at 106.68 29.21 0)
 			(show_name no)
 			(do_not_autoplace no)
@@
 			)
 		)
-		(property "Footprint" "wsprrypi-zero-gpio-bs170:C_0603_1608Metric"
+		(property "Footprint" "wsprrypi-zero-gpio-bs170:C_1206_3216Metric"
 			(at 106.68 26.67 0)
 			(hide yes)
@@
 			)
 		)
-		(property "Datasheet" "https://www.lcsc.com/datasheet/C235731.pdf"
+		(property "Datasheet" "https://www.lcsc.com/datasheet/C170182.pdf?spm=wm.sxq.inf.ggs&lcsc_vid=RgUIVQJUTldWUAAER1JWUgUFQAdWUVZWEgRWUAJSRVYxVlNfRlNeXlxSRVVZVztW"
 			(at 106.68 26.67 0)
 			(hide yes)
@@
 			)
 		)
-		(property "Description" "CAP CER 100nF ±10% 50V X7R 0603"
+		(property "Description" "CAP CER 100nF 50V NP0 1206"
 			(at 106.68 26.67 0)
 			(hide yes)
@@
 			)
 		)
-		(property "Manufacturer" "PSA"
+		(property "Manufacturer" "Walsin"
 			(at 106.68 26.67 0)
 			(hide yes)
@@
 			)
 		)
-		(property "MPN" "FN18X104K500PBG"
+		(property "MPN" "1206N104J500CT"
 			(at 106.68 26.67 0)
 			(hide yes)
@@
 			)
 		)
-		(property "LCSC_PART" "C235731"
+		(property "LCSC Part #" "C170182"
 			(at 106.68 26.67 0)
 			(hide yes)
@@
 		(in_bom no)
 		(on_board yes)
-		(in_pos_files yes)
+		(in_pos_files no)
 		(dnp no)
 		(property "Reference" "J51"
@@
 			)
 		)
-		(property "LCSC_PART" "C25803"
+		(property "LCSC Part #" "C25803"
 			(at 120.65 31.75 0)
 			(hide yes)
@@
 			)
 		)
-		(property "LCSC_PART" "C2286"
+		(property "LCSC Part #" "C2286"
 			(at 76.2 96.52 0)
 			(hide yes)
@@
 			)
 		)
-		(property "LCSC_PART" "C726584"
+		(property "LCSC Part #" "C726584"
 			(at 148.59 82.55 0)
 			(hide yes)
@@
 			)
 		)
-		(property "LCSC_PART" "C726584"
+		(property "LCSC Part #" "C726584"
 			(at 166.37 22.86 0)
 			(hide yes)
@@
 			)
 		)
-		(property "LCSC_PART" "C20070397"
+		(property "LCSC Part #" "C20070397"
 			(at 102.87 82.55 0)
 			(hide yes)
@@
 			)
 		)
-		(property "LCSC_PART" "C23162"
+		(property "LCSC Part #" "C23162"
 			(at 125.73 45.72 0)
 			(hide yes)
@@
 	)
 	(symbol
-		(lib_id "wsprrypi-zero-gpio-bs170:R_0805")
+		(lib_id "wsprrypi-zero-gpio-bs170:R_0805_0R_Jumper")
 		(at 156.21 21.59 0)
 		(unit 1)
@@
 			)
 		)
-		(property "LCSC_PART" "C2907288"
+		(property "LCSC Part #" "C2907288"
 			(at 156.21 21.59 0)
 			(hide yes)
@@
 			)
 		)
-		(property "LCSC_PART" "C1588"
+		(property "LCSC Part #" "C1588"
 			(at 129.54 90.17 0)
 			(hide yes)
@@
 			)
 		)
-		(property "LCSC_PART" "C131941"
+		(property "LCSC Part #" "C131941"
 			(at 116.84 86.36 0)
 			(hide yes)
@@
 			)
 		)
-		(property "LCSC_PART" "C2907014"
+		(property "LCSC Part #" "C2907014"
 			(at 67.31 96.52 90)
 			(hide yes)
@@
 			)
 		)
-		(property "LCSC_PART" "C719177"
+		(property "LCSC Part #" "C719177"
 			(at 110.49 50.8 0)
 			(hide yes)
@@
 			)
 		)
-		(property "LCSC_PART" "C25803"
+		(property "LCSC Part #" "C25803"
 			(at 102.87 92.71 90)
 			(hide yes)
@@
 	)
 	(symbol
-		(lib_id "wsprrypi-zero-gpio-bs170:C_0603")
-		(at 181.61 80.01 0)
-		(mirror x)
-		(unit 1)
-		(body_style 1)
-		(exclude_from_sim no)
-		(in_bom yes)
-		(on_board yes)
-		(in_pos_files yes)
-		(dnp no)
-		(property "Reference" "C51"
-			(at 181.61 85.09 0)
-			(show_name no)
-			(do_not_autoplace no)
-			(effects
-				(font
-					(size 1.27 1.27)
-				)
-			)
-		)
-		(property "Value" "100nF"
-			(at 181.61 82.55 0)
-			(show_name no)
-			(do_not_autoplace no)
-			(effects
-				(font
-					(size 1.27 1.27)
-				)
-			)
-		)
-		(property "Footprint" "wsprrypi-zero-gpio-bs170:C_0603_1608Metric"
-			(at 181.61 80.01 0)
-			(hide yes)
-			(show_name no)
-			(do_not_autoplace no)
-			(effects
-				(font
-					(size 1.27 1.27)
-				)
-			)
-		)
-		(property "Datasheet" "https://www.lcsc.com/datasheet/C235731.pdf"
-			(at 181.61 80.01 0)
-			(hide yes)
-			(show_name no)
-			(do_not_autoplace no)
-			(effects
-				(font
-					(size 1.27 1.27)
-				)
-			)
-		)
-		(property "Description" "CAP CER 100nF ±10% 50V X7R 0603"
-			(at 181.61 80.01 0)
-			(hide yes)
-			(show_name no)
-			(do_not_autoplace no)
-			(effects
-				(font
-					(size 1.27 1.27)
-				)
-			)
-		)
-		(property "Manufacturer" "PSA"
-			(at 181.61 80.01 0)
-			(hide yes)
-			(show_name no)
-			(do_not_autoplace no)
-			(effects
-				(font
-					(size 1.27 1.27)
-				)
-			)
-		)
-		(property "MPN" "FN18X104K500PBG"
-			(at 181.61 80.01 0)
-			(hide yes)
-			(show_name no)
-			(do_not_autoplace no)
-			(effects
-				(font
-					(size 1.27 1.27)
-				)
-			)
-		)
-		(property "LCSC_PART" "C235731"
-			(at 181.61 80.01 0)
-			(hide yes)
-			(show_name no)
-			(do_not_autoplace no)
-			(effects
-				(font
-					(size 1.27 1.27)
-				)
-			)
-		)
-		(pin "1"
-		)
-		(pin "2"
-		)
-		(instances
-			(project "WsprryPi Zero GPIO BS170"
-				(path "/42fb2efa-c288-4686-a90a-043ad23a327d"
-					(reference "C51")
-					(unit 1)
-				)
-			)
-		)
-	)
-	(symbol
 		(lib_id "wsprrypi-zero-gpio-bs170:Conn_01x03")
 		(at 76.2 64.77 90)
@@
 			)
 		)
-		(property "LCSC_PART" "C2907002"
+		(property "LCSC Part #" "C2907002"
 			(at 138.43 86.36 0)
 			(hide yes)
@@
 	)
 	(symbol
+		(lib_id "wsprrypi-zero-gpio-bs170:C_0603")
+		(at 181.61 80.01 0)
+		(mirror x)
+		(unit 1)
+		(body_style 1)
+		(exclude_from_sim no)
+		(in_bom yes)
+		(on_board yes)
+		(in_pos_files yes)
+		(dnp no)
+		(property "Reference" "C51"
+			(at 181.61 77.47 0)
+			(show_name no)
+			(do_not_autoplace no)
+			(effects
+				(font
+					(size 1.27 1.27)
+				)
+			)
+		)
+		(property "Value" "100nF"
+			(at 181.61 82.55 0)
+			(show_name no)
+			(do_not_autoplace no)
+			(effects
+				(font
+					(size 1.27 1.27)
+				)
+			)
+		)
+		(property "Footprint" "wsprrypi-zero-gpio-bs170:C_1206_3216Metric"
+			(at 181.61 80.01 0)
+			(hide yes)
+			(show_name no)
+			(do_not_autoplace no)
+			(effects
+				(font
+					(size 1.27 1.27)
+				)
+			)
+		)
+		(property "Datasheet" "https://www.lcsc.com/datasheet/C170182.pdf?spm=wm.sxq.inf.ggs&lcsc_vid=RgUIVQJUTldWUAAER1JWUgUFQAdWUVZWEgRWUAJSRVYxVlNfRlNeXlxSRVVZVztW"
+			(at 181.61 80.01 0)
+			(hide yes)
+			(show_name no)
+			(do_not_autoplace no)
+			(effects
+				(font
+					(size 1.27 1.27)
+				)
+			)
+		)
+		(property "Description" "CAP CER 100nF 50V NP0 1206"
+			(at 181.61 80.01 0)
+			(hide yes)
+			(show_name no)
+			(do_not_autoplace no)
+			(effects
+				(font
+					(size 1.27 1.27)
+				)
+			)
+		)
+		(property "Manufacturer" "Walsin"
+			(at 181.61 80.01 0)
+			(hide yes)
+			(show_name no)
+			(do_not_autoplace no)
+			(effects
+				(font
+					(size 1.27 1.27)
+				)
+			)
+		)
+		(property "MPN" "1206N104J500CT"
+			(at 181.61 80.01 0)
+			(hide yes)
+			(show_name no)
+			(do_not_autoplace no)
+			(effects
+				(font
+					(size 1.27 1.27)
+				)
+			)
+		)
+		(property "LCSC Part #" "C170182"
+			(at 181.61 80.01 0)
+			(hide yes)
+			(show_name no)
+			(do_not_autoplace no)
+			(effects
+				(font
+					(size 1.27 1.27)
+				)
+			)
+		)
+		(pin "1"
+		)
+		(pin "2"
+		)
+		(instances
+			(project "WsprryPi Zero GPIO BS170"
+				(path "/42fb2efa-c288-4686-a90a-043ad23a327d"
+					(reference "C51")
+					(unit 1)
+				)
+			)
+		)
+	)
+	(symbol
 		(lib_id "wsprrypi-zero-gpio-bs170:GND")
 		(at 161.29 54.61 0)
@@
 			)
 		)
-		(property "LCSC_PART" "C470426"
+		(property "LCSC Part #" "C470426"
 			(at 22.86 97.79 0)
 			(hide yes)
