File: WsprryPico Shield/WsprryPico Shield.kicad_pcb (KiCad board)
At the start: 2 copper layers, 53.3 x 22.9 mm, 1 part

Commit message: Finish Pick BS170 design
Parts:
- added C21: 10µF, wsprrypico-shield:C_0805_2012Metric, B.Cu at (121.4, 83.5)
- added C22: 1nF, wsprrypico-shield:C_0603_1608Metric, B.Cu at (127.2, 85.0)
- added C23: 1µF, wsprrypico-shield:C_0805_2012Metric, B.Cu at (128.1, 87.4)
- added C31: 100nF, wsprrypico-shield:C_1206_3216Metric, B.Cu at (131.2, 96.3)
- added C32: 100nF, wsprrypico-shield:C_0603_1608Metric, B.Cu at (148.9, 95.2)
- added C41: 100nF, wsprrypico-shield:C_0603_1608Metric, B.Cu at (143.9, 90.4)
- added C42: 1µF, wsprrypico-shield:C_0805_2012Metric, B.Cu at (146.4, 90.9)
- added C51: 100nF, wsprrypico-shield:C_1206_3216Metric, B.Cu at (127.7, 92.2)
- added D11: KT-0603R, wsprrypico-shield:LED_0603_1608Metric, B.Cu at (135.9, 82.8)
- added J51: SMA_Adafruit_1865, wsprrypico-shield:SMA_Adafruit_1865_EdgeMount, B.Cu at (121.8, 94.1)
- added JP1: BIAS, Jumper:SolderJumper-2_P1.3mm_Open_RoundedPad1.0x1.5mm, B.Cu at (124.4, 87.5)
- added L41: 25T FT37-43, wsprrypico-shield:L_Toroid_FT37-43_Vertical_P5.08mm, B.Cu at (141.6, 91.2)
- added Q41: BS170, wsprrypico-shield:TO-92_Inline, B.Cu at (131.6, 91.2)
- added R11: 220Ω, wsprrypico-shield:R_0603_1608Metric, B.Cu at (132.9, 82.8)
- added R21: 100kΩ, wsprrypico-shield:R_0603_1608Metric, B.Cu at (127.2, 82.5)
- added R22: 1kΩ, wsprrypico-shield:R_0603_1608Metric, B.Cu at (126.4, 87.2)
- added R31: 22Ω, wsprrypico-shield:R_0603_1608Metric, B.Cu at (128.2, 96.0)
- added R32: 4.7kΩ, wsprrypico-shield:R_0603_1608Metric, B.Cu at (143.8, 95.8)
- added R33: 100kΩ, wsprrypico-shield:R_0603_1608Metric, B.Cu at (134.3, 93.3)
- added RV31: 5kΩ, wsprrypico-shield:Potentiometer_Bourns_TC33X_Vertical, B.Cu at (146.4, 94.5)
- added U21: TPS22918DBVR, wsprrypico-shield:SOT-23-6, B.Cu at (124.0, 83.8)
- renumbered U1 to U11
Connections:
- U11 pad 13: unconnected-(U1-GND-Pad13) -> GND
- U11 pad 18: unconnected-(U1-GND-Pad18) -> GND
- U11 pad 20: unconnected-(U1-GP15-Pad20) -> /AMP_EN
- U11 pad 23: unconnected-(U1-GND-Pad23) -> GND
- U11 pad 28: unconnected-(U1-GND-Pad28) -> GND
- U11 pad 29: unconnected-(U1-GP22-Pad29) -> /PICO_LED
- U11 pad 3: unconnected-(U1-GND-Pad3) -> GND
- U11 pad 38: unconnected-(U1-GND-Pad38) -> GND
- U11 pad 4: unconnected-(U1-GP2-Pad4) -> /PICO_RF
- U11 pad 40: unconnected-(U1-VBUS-Pad40) -> /AMP_5V_IN
- U11 pad 8: unconnected-(U1-GND-Pad8) -> GND
Routing:
- net /AMP_EN: track 0.00 -> 53.3 mm
- net /SW_5V: track 0.00 -> 35.4 mm
- net /GATE: track 0.00 -> 21.1 mm
- net GND: track 0.00 -> 18.9 mm, vias 0 -> 19
- net /PICO_LED: track 0.00 -> 14.7 mm
- net /AMP_5V_IN: track 0.00 -> 13.1 mm
- net /PA_DRAIN: track 0.00 -> 8.98 mm
- net Net-(C32-Pad2): track 0.00 -> 5.58 mm
- net /PICO_RF: track 0.00 -> 4.13 mm
- net /FINAL_OUT: track 0.00 -> 3.83 mm
- net Net-(U21-QOD): track 0.00 -> 3.30 mm
- net Net-(C31-Pad2): track 0.00 -> 1.76 mm
- net Net-(U21-CT): track 0.00 -> 1.46 mm
- net Net-(D11-K): track 0.00 -> 1.34 mm
- added copper zone on F.Cu, net GND
