File: WsprryPico Shield/WsprryPico Shield.kicad_sch (KiCad schematic)
At the start: 3 parts, among them J1 Socket_1x20_P2.54mm, J2 Socket_1x20_P2.54mm

Commit message: Finish Pick BS170 design
Parts:
- added C21: 10µF, wsprrypico-shield:C_0805_2012Metric, symbol wsprrypico-shield:C_0805
- added C22: 1nF, wsprrypico-shield:C_0603_1608Metric, symbol wsprrypico-shield:C_0603
- added C23, C42: 1µF, wsprrypico-shield:C_0805_2012Metric, symbol wsprrypico-shield:C_0805
- added C31, C51: 100nF, wsprrypico-shield:C_1206_3216Metric, symbol wsprrypico-shield:C_0603
- added C32, C41: 100nF, wsprrypico-shield:C_0603_1608Metric, symbol wsprrypico-shield:C_0603
- added D11: KT-0603R, wsprrypico-shield:LED_0603_1608Metric, symbol wsprrypico-shield:LED
- added J51: SMA_Adafruit_1865, wsprrypico-shield:SMA_Adafruit_1865_EdgeMount, symbol wsprrypico-shield:SMA_Adafruit_1865
- added JP1: BIAS, Jumper:SolderJumper-2_P1.3mm_Open_RoundedPad1.0x1.5mm, symbol Jumper:SolderJumper_2_Open
- added L41: 25T FT37-43, wsprrypico-shield:L_Toroid_FT37-43_Vertical_P5.08mm, symbol wsprrypico-shield:L
- added Q41: BS170, wsprrypico-shield:TO-92_Inline, symbol wsprrypico-shield:BS170
- added R11: 220Ω, wsprrypico-shield:R_0603_1608Metric, symbol wsprrypico-shield:R_US
- added R21, R33: 100kΩ, wsprrypico-shield:R_0603_1608Metric, symbol wsprrypico-shield:R_0603
- added R22: 1kΩ, wsprrypico-shield:R_0603_1608Metric, symbol wsprrypico-shield:R_0603
- added R31: 22Ω, wsprrypico-shield:R_0603_1608Metric, symbol wsprrypico-shield:R_0603
- added R32: 4.7kΩ, wsprrypico-shield:R_0603_1608Metric, symbol wsprrypico-shield:R_0603
- added RV31: 5kΩ, wsprrypico-shield:Potentiometer_Bourns_TC33X_Vertical, symbol wsprrypico-shield:R_Potentiometer_US
- added U21: TPS22918DBVR, wsprrypico-shield:SOT-23-6, symbol wsprrypico-shield:TPS22918
- renumbered J1 to J11, J2 to J12, U1 to U11
Connections:
- net GND: now reaches U11.13 (GND)
- net GND: now also U11.18 (GND), U11.23 (GND), U11.28 (GND), U11.3 (GND), U11.38 (GND), U11.8 (GND), C21.2, C22.2, C23.2, C32.1, C41.2, C42.2, J51.2 (GND), Q41.3 (S), R11.2, R21.2, R33.1, RV31.3, U21.2 (GND)
- net AMP_EN: now reaches U11.20 (GP15)
- net AMP_EN: now also R21.1, U21.3 (ON)
- net PICO_LED: now reaches U11.29 (GP22)
- net PICO_LED: now also D11.2 (A)
- net PICO_RF: now reaches U11.4 (GP2)
- net PICO_RF: now also C31.1
- net AMP_5V_IN: now reaches U11.40 (VBUS)
- net AMP_5V_IN: now also C21.1, JP1.1 (A), U21.1 (VIN)
- new net: C32.2, R32.1, RV31.2
- new net: D11.1 (K), R11.1
- new net: C22.1, U21.4 (CT)
- new net: R22.2, U21.5 (QOD)
- new net: C31.2, R31.1
- new net FINAL_OUT: C51.2, J51.1 (In)
- new net GATE: Q41.2 (G), R31.2, R32.2, R33.2
- new net PA_DRAIN: C51.1, L41.2, Q41.1 (D)
- new net SW_5V: C23.1, C41.1, C42.1, JP1.2 (B), L41.1, R22.1, RV31.1, U21.6 (VOUT)
- no-connect marks 0 -> 29
Other:
- note added: "BIAS SET - normally open"
- note added: "Pico interface: J11 / J12 sockets (purchasing only)"
- note removed: "Pico interface: two female sockets (BOM only)"
- note removed: "Starter interface: pins are intentionally unwired. Wire required pins; mark only unused pins with no-connect flags. J1 + J2 describe the sockets; excluded from BOM and placement."
- company: (none) -> Lee Bussy [AA0NT]
- title: (none) -> WsprryPico Shield - BS170 circuit, Pico bus open
- moved on the sheet: J11, J12, U11
