File: WsprryPico Synth Shield/WsprryPico Synth Shield.kicad_sch (KiCad schematic)
At the start: 3 parts, among them J11 Socket_1x20_P2.54mm, J12 Socket_1x20_P2.54mm

Commit message: Specify synth shield parts and place decade-series symbols
Parts:
- added C21, C81: 10nF X7R, wsprrypico-synth-shield:C_0603_1608Metric, symbol wsprrypico-synth-shield:C
- added C22, C52: 1nF C0G, wsprrypico-synth-shield:C_0603_1608Metric, symbol wsprrypico-synth-shield:C
- added C23, C31, C32, C54, C62, C71, C73: 100nF X7R, wsprrypico-synth-shield:C_0603_1608Metric, symbol wsprrypico-synth-shield:C
- added C41, C42, C74: 2.2uF X7R, wsprrypico-synth-shield:C_0805_2012Metric, symbol wsprrypico-synth-shield:C
- added C51: 10uF X7R, wsprrypico-synth-shield:C_1206_3216Metric, symbol wsprrypico-synth-shield:C
- added C53, C63, C72: 1uF X7R, wsprrypico-synth-shield:C_0805_2012Metric, symbol wsprrypico-synth-shield:C
- added C61, C64: 100nF C0G, wsprrypico-synth-shield:C_1206_3216Metric, symbol wsprrypico-synth-shield:C
- added D81: Red, wsprrypico-synth-shield:LED_0603_1608Metric, symbol wsprrypico-synth-shield:LED
- added J61: SMA 50ohm, wsprrypico-synth-shield:SMA_BAT_Wireless_BWSMA-KWE-Z001, symbol wsprrypico-synth-shield:SMA
- added J71: GPS PH-5, wsprrypico-synth-shield:JST_PH_B5B-PH-K_1x05_P2.00mm_Vertical, symbol wsprrypico-synth-shield:Conn_01x05
- added JP41: VBUS default, wsprrypico-synth-shield:PowerSelector_VBUS_IN_VSYS_Cuttable, symbol wsprrypico-synth-shield:PowerSelector
- added JP51: Normally open, wsprrypico-synth-shield:SolderJumper-2_P1.3mm_Open_RoundedPad1.0x1.5mm, symbol wsprrypico-synth-shield:SolderJumper_2_Open
- added L61: 25T FT37-43, wsprrypico-synth-shield:L_Toroid_FT37-43_Vertical_P5.08mm, symbol wsprrypico-synth-shield:L
- added Q61: BS170, wsprrypico-synth-shield:TO-92_Inline, symbol wsprrypico-synth-shield:BS170
- added R31, R32, R62: 4.7k, wsprrypico-synth-shield:R_0603_1608Metric, symbol wsprrypico-synth-shield:R
- added R51, R63, R73: 100k, wsprrypico-synth-shield:R_0603_1608Metric, symbol wsprrypico-synth-shield:R
- added R52, R75, R82, R83: 1k, wsprrypico-synth-shield:R_0603_1608Metric, symbol wsprrypico-synth-shield:R
- added R61: 22R, wsprrypico-synth-shield:R_0603_1608Metric, symbol wsprrypico-synth-shield:R
- added R71, R72, R81: 10k, wsprrypico-synth-shield:R_0603_1608Metric, symbol wsprrypico-synth-shield:R
- added R74: 33R, wsprrypico-synth-shield:R_0603_1608Metric, symbol wsprrypico-synth-shield:R
- added RV61: 5k, wsprrypico-synth-shield:Potentiometer_Bourns_TC33X_Vertical, symbol wsprrypico-synth-shield:R_Potentiometer_US
- added SW81: Push, wsprrypico-synth-shield:SW_SPST_XUNPU_TS1088R_4x3mm, symbol wsprrypico-synth-shield:SW_Push
- added U31: Si5351A-B-GTR, wsprrypico-synth-shield:MSOP-10_Si5351A_3x3mm_P0.5mm, symbol wsprrypico-synth-shield:Si5351A
- added U41: TPS7A2033, wsprrypico-synth-shield:SOT-23-5, symbol wsprrypico-synth-shield:TPS7A2033PDBVR
- added U51: TPS22918, wsprrypico-synth-shield:SOT-23-6, symbol wsprrypico-synth-shield:TPS22918
- added U71: LS7366R-S, wsprrypico-synth-shield:SOIC-14_3.9x8.7mm_P1.27mm, symbol wsprrypico-synth-shield:LS7366R_S
- added U72: SN74LVC1G14, wsprrypico-synth-shield:SOT-23-5, symbol wsprrypico-synth-shield:SN74LVC1G14DBVR
- added Y21: 25MHz TCXO, wsprrypico-synth-shield:KDS_DSB321SDN_3.2x2.5mm, symbol wsprrypico-synth-shield:KDS_DSB321SDN_25MHz
- J11, J12: value Socket_1x20_P2.54mm -> 1x20 socket; Assembly (none) -> Manual; Board interface (none) -> U11 combined 40-pad footprint; Function (none) -> Pico female socket; purchased separately; PCB pads belong t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; LCSC Part # (none) -> C5224030; MPN (none) -> PM2.54-1*20; Manufacturer (none) -> ZHOURI; Rating (none) -> 2.5 A nominal; Selection status (none) -> Selected prototype; Specified Value (none) -> 1x20; 2.54 mm; 8.5 mm body; Supplier URL (none) -> https://www.lcsc.com/product-detail/C5224030.html; Technology (none) -> PBT; Au over Ni; Tolerance (none) -> Drawing dimensions
Other:
- note added: "GPS header: 1 3V3 / 2 GND / 3 GPS_TX / 4 GPS_RX / 5 PPS"
- note added: "L61 hand-wound: no BOM / positions; source pending. Output DC block -> SMA -> external LPF."
- note added: "Manual sockets: no BOM / positions"
- note added: "Placement only: connections and PCB synchronization are pending. Always-on clock; independent AMP_EN. GP6 / GP14 / GP15 remain unapproved control candidates."
- note removed: "Pico interface: two female sockets (BOM only)"
- note removed: "Starter interface: pins are intentionally unwired. Wire required pins; mark only unused pins with no-connect flags. J11 + J12 describe the sockets; excluded from BOM and placement."
- title: (none) -> WsprryPico Synth Shield
- moved on the sheet: J11, J12, U11

Commit message: Add QLG3 receiver assembly and assign plain-header J71
Parts:
- J71: value GPS PH-5 -> QLG3 GPS Receiver; footprint wsprrypico-synth-shield:JST_PH_B5B-PH-K_1x05_P2.00mm_Vertical -> wsprrypico-synth-shield:QLG3_GPS_UndersideHeader; Function External optional GPS interface -> QLG3 GPS Receiver with shield-top socket and downward matin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; LCSC Part # C157993 -> (none); MPN B5B-PH-K-S(LF)(SN) -> QLG3; standard 1x05 2.54 mm socket/header; Manufacturer JST -> QRP Labs module; generic unkeyed mating headers; Rating 3.3 V signals and power -> 3.3 V power; QLG3 2.8 V UART/PPS outputs; Selection status Selected prototype -> Standard pitch and QLG3 footprint selected; final mating ha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; Specified Value JST PH 5-way; 2.0 mm; top entry -> 1x05 female socket and male header; 0.1 inch (2.54 mm); unk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; Supplier URL https://www.lcsc.com/product-detail/C157993.html -> https://qrp-labs.com/qlg3.html; Technology Keyed connector -> Unkeyed through-hole pin socket/header
Other:
- note added: "QLG3 header: 1 3V3 / 2 VBAT(3V3) / 3 PPS / 4 GPS_TX / 5 GND"
- note removed: "GPS header: 1 3V3 / 2 GND / 3 GPS_TX / 4 GPS_RX / 5 PPS"
Changed lines of the file:
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@@
 (lib_id "wsprrypico-synth-shield:Conn_01x05") (at 387.35 163.83 0) (unit 1) (body_style 1) (exclude_from_sim no) (in_bom no) (on_board yes) (in_pos_files no) (dnp no)
 (property "Reference" "J71" (at 382.27 154.94 0) (show_name no) (do_not_autoplace no) (effects (font (size 1.27 1.27))))
-(property "Value" "GPS PH-5" (at 382.27 172.72 0) (show_name no) (do_not_autoplace no) (effects (font (size 1.27 1.27))))
-(property "Footprint" "wsprrypico-synth-shield:JST_PH_B5B-PH-K_1x05_P2.00mm_Vertical" (at 387.35 163.83 0) (show_name no) (do_not_autoplace no) (hide yes) (effects (font (size 1.27 1.27))))
-(property "Datasheet" "https://www.jst-mfg.com/product/pdf/eng/ePH.pdf" (at 387.35 163.83 0) (show_name no) (do_not_autoplace no) (hide yes) (effects (font (size 1.27 1.27))))
-(property "Description" "External optional GPS interface; JST PH 5-way; 2.0 mm; top entry; Keyed connector" (at 387.35 163.83 0) (show_name no) (do_not_autoplace no) (hide yes) (effects (font (size 1.27 1.27))))
-(property "Manufacturer" "JST" (at 387.35 163.83 0) (show_name no) (do_not_autoplace no) (hide yes) (effects (font (size 1.27 1.27))))
-(property "MPN" "B5B-PH-K-S(LF)(SN)" (at 387.35 163.83 0) (show_name no) (do_not_autoplace no) (hide yes) (effects (font (size 1.27 1.27))))
-(property "LCSC Part #" "C157993" (at 387.35 163.83 0) (show_name no) (do_not_autoplace no) (hide yes) (effects (font (size 1.27 1.27))))
-(property "Supplier URL" "https://www.lcsc.com/product-detail/C157993.html" (at 387.35 163.83 0) (show_name no) (do_not_autoplace no) (hide yes) (effects (font (size 1.27 1.27))))
-(property "Specified Value" "JST PH 5-way; 2.0 mm; top entry" (at 387.35 163.83 0) (show_name no) (do_not_autoplace no) (hide yes) (effects (font (size 1.27 1.27))))
-(property "Technology" "Keyed connector" (at 387.35 163.83 0) (show_name no) (do_not_autoplace no) (hide yes) (effects (font (size 1.27 1.27))))
+(property "Value" "QLG3 GPS Receiver" (at 382.27 172.72 0) (show_name no) (do_not_autoplace no) (effects (font (size 1.27 1.27))))
+(property "Footprint" "wsprrypico-synth-shield:QLG3_GPS_UndersideHeader" (at 387.35 163.83 0) (show_name no) (do_not_autoplace no) (hide yes) (effects (font (size 1.27 1.27))))
+(property "Datasheet" "https://qrp-labs.com/qlg3.html" (at 387.35 163.83 0) (show_name no) (do_not_autoplace no) (hide yes) (effects (font (size 1.27 1.27))))
+(property "Description" "QRP Labs QLG3 GPS Receiver; plain 1x5 0.1-inch (2.54 mm) socket/header; full receiver assembly model" (at 387.35 163.83 0) (show_name no) (do_not_autoplace no) (hide yes) (effects (font (size 1.27 1.27))))
+(property "Manufacturer" "QRP Labs module; generic unkeyed mating headers" (at 387.35 163.83 0) (show_name no) (do_not_autoplace no) (hide yes) (effects (font (size 1.27 1.27))))
+(property "MPN" "QLG3; standard 1x05 2.54 mm socket/header" (at 387.35 163.83 0) (show_name no) (do_not_autoplace no) (hide yes) (effects (font (size 1.27 1.27))))
+(property "LCSC Part #" "" (at 387.35 163.83 0) (show_name no) (do_not_autoplace no) (hide yes) (effects (font (size 1.27 1.27))))
+(property "Supplier URL" "https://qrp-labs.com/qlg3.html" (at 387.35 163.83 0) (show_name no) (do_not_autoplace no) (hide yes) (effects (font (size 1.27 1.27))))
+(property "Specified Value" "1x05 female socket and male header; 0.1 inch (2.54 mm); unkeyed" (at 387.35 163.83 0) (show_name no) (do_not_autoplace no) (hide yes) (effects (font (size 1.27 1.27))))
+(property "Technology" "Unkeyed through-hole pin socket/header" (at 387.35 163.83 0) (show_name no) (do_not_autoplace no) (hide yes) (effects (font (size 1.27 1.27))))
 (property "Tolerance" "Drawing dimensions" (at 387.35 163.83 0) (show_name no) (do_not_autoplace no) (hide yes) (effects (font (size 1.27 1.27))))
-(property "Rating" "3.3 V signals and power" (at 387.35 163.83 0) (show_name no) (do_not_autoplace no) (hide yes) (effects (font (size 1.27 1.27))))
+(property "Rating" "3.3 V power; QLG3 2.8 V UART/PPS outputs" (at 387.35 163.83 0) (show_name no) (do_not_autoplace no) (hide yes) (effects (font (size 1.27 1.27))))
 (property "Assembly" "Manual" (at 387.35 163.83 0) (show_name no) (do_not_autoplace no) (hide yes) (effects (font (size 1.27 1.27))))
-(property "Function" "External optional GPS interface" (at 387.35 163.83 0) (show_name no) (do_not_autoplace no) (hide yes) (effects (font (size 1.27 1.27))))
-(property "Selection status" "Selected prototype" (at 387.35 163.83 0) (show_name no) (do_not_autoplace no) (hide yes) (effects (font (size 1.27 1.27))))
+(property "Function" "QLG3 GPS Receiver with shield-top socket and downward mating pins" (at 387.35 163.83 0) (show_name no) (do_not_autoplace no) (hide yes) (effects (font (size 1.27 1.27))))
+(property "Selection status" "Standard pitch and QLG3 footprint selected; final mating hardware fit pending" (at 387.35 163.83 0) (show_name no) (do_not_autoplace no) (hide yes) (effects (font (size 1.27 1.27))))
 (pin "1")
 (pin "2")
@@
 	(text "Manual sockets: no BOM / positions" (exclude_from_sim no) (at 60.96 120.65 0) (effects (font (size 1.27 1.27)) ))
 	(text "L61 hand-wound: no BOM / positions; source pending.\nOutput DC block -> SMA -> external LPF." (exclude_from_sim no) (at 120.65 242.57 0) (effects (font (size 1.27 1.27)) (justify left)))
-	(text "GPS header: 1 3V3 / 2 GND / 3 GPS_TX / 4 GPS_RX / 5 PPS" (exclude_from_sim no) (at 264.16 248.92 0) (effects (font (size 1.27 1.27)) (justify left)))
+	(text "QLG3 header: 1 3V3 / 2 VBAT(3V3) / 3 PPS / 4 GPS_TX / 5 GND" (exclude_from_sim no) (at 264.16 248.92 0) (effects (font (size 1.27 1.27)) (justify left)))
 	(text "Placement only: connections and PCB synchronization are pending.\nAlways-on clock; independent AMP_EN. GP6 / GP14 / GP15 remain unapproved control candidates." (exclude_from_sim no) (at 12.7 269.24 0) (effects (font (size 1.27 1.27)) (justify left)))
 )

Commit message: Set up schematic
Parts:
- removed C54: 100nF X7R, wsprrypico-synth-shield:C_0603_1608Metric, symbol wsprrypico-synth-shield:C
- added C65: 100nF, wsprrypico-synth-shield:C_0603_1608Metric, symbol wsprrypico-synth-shield:C
- added TP71: GPS_RX, wsprrypico-synth-shield:TestPoint_Pad_D2.0mm, symbol wsprrypico-synth-shield:TestPoint
- C21, C81: value 10nF X7R -> 10nF
- C23, C31, C32, C62, C71, C73: value 100nF X7R -> 100nF
- C41, C42, C74: value 2.2uF X7R -> 2.2μF
- C51: value 10uF X7R -> 10μF
- C52: value 1nF C0G -> 1nF
- C53, C63, C72: value 1uF X7R -> 1μF
- C61, C64: value 100nF C0G -> 100nF
- JP41: value VBUS default -> SolderJumper_3_Bridged12; symbol wsprrypico-synth-shield:PowerSelector -> wsprrypico-synth-shield:SolderJumper_3_Bridged12
- JP51: value Normally open -> BIAS_SET
- R31, R32, R62: value 4.7k -> 4.7kΩ
- R51, R63, R73: value 100k -> 100kΩ
- R52, R75, R82, R83: value 1k -> 1kΩ
- R61: value 22R -> 22Ω
- R71, R72, R81: value 10k -> 10kΩ
- R74: value 33R -> 33Ω
- RV61: value 5k -> 5kΩ
Connections:
- net SYNTH_3V3: now reaches C32.1
- net SYNTH_3V3: now also C21.1, C23.1, C31.1, C42.1, R31.1, R32.1, U31.1 (VDD), U31.7 (VDDO), U41.5 (OUT), Y21.4 (VCC)
- net GND: now reaches C32.2
- net GND: now also C21.2, C23.2, C31.2, C41.2, C42.2, C51.2, C52.2, C53.2, C62.2, C63.2, C71.2, C72.2, C73.2, C74.2, C81.2, D81.1 (K), J61.2 (GND), J71.5 (Pin_5), Q61.3 (S), R51.2, R63.2, R73.2, RV61.3, SW81.2, U11.13 (GND), U11.18 (GND), U11.23 (GND), U11.28 (GND), U11.3 (GND), U11.33 (AGND), U11.38 (GND), U11.8 (GND), U31.8 (GND), U41.2 (GND), U51.2 (GND), U71.2 (fCKi), U71.3 (VSS), U72.3 (GND), Y21.1 (GND), Y21.2 (GND), C65.2
- net at C22.1: now also Y21.3 (OUT)
- net XA: now reaches C22.2
- net XA: now also U31.2 (XA)
- net GPS_PPS: now reaches R73.1
- net GPS_PPS: now also R75.2, U11.21 (GP16), U72.2
- net PICO_3V3: now reaches C73.1
- net PICO_3V3: now also C71.1, C72.1, C74.1, J71.1 (Pin_1), J71.2 (Pin_2), R71.1, R72.1, R81.1, U11.36 (3V3_OUT), U71.11 (B), U71.13 (CNT_EN), U71.14 (VDD), U72.5 (VCC)
- net COUNTER_INDEX_N: now reaches U71.10 (~{INDEX})
- net COUNTER_INDEX_N: now also U72.4
- net COUNTER_CLK: now reaches U71.12 (A)
- net COUNTER_CLK: now also R74.2
- net COUNTER_CS_N: now reaches U71.4 (~{SS})
- net COUNTER_CS_N: now also R71.2, U11.17 (GP13)
- net COUNTER_SCK: now reaches U71.5 (SCK)
- net COUNTER_SCK: now also U11.14 (GP10)
- net COUNTER_MISO: now reaches U71.6 (MISO)
- net COUNTER_MISO: now also U11.16 (GP12)
- net COUNTER_MOSI: now reaches U71.7 (MOSI)
- net COUNTER_MOSI: now also U11.15 (GP11)
- net COUNTER_IRQ_N: now reaches U71.8 (~{LFLAG})
- net COUNTER_IRQ_N: now also R72.2, U11.22 (GP17)
- net BUTTON_SW: now reaches C81.1
- net BUTTON_SW: now also R81.2, R83.1, SW81.1
- net LED_A: now reaches D81.2 (A)
- net LED_A: now also R82.2
- net AMP_5V_SW: now reaches C63.1
- net AMP_5V_SW: now also C53.1, C62.1, JP51.2 (B), L61.1, R52.2, RV61.1, U51.6 (VOUT)
- net SYNTH_CLK2: now reaches R74.1
- net SYNTH_CLK2: now also U31.6 (CLK2)
- net LED_DRIVE: now reaches R82.1
- net LED_DRIVE: now also U11.20 (GP15)
- net SYNTH_SDA: now reaches R31.2
- net SYNTH_SDA: now also U11.6 (GP4), U31.5 (SDA)
- net GPS_RX: now reaches U11.1 (GP0)
- net GPS_RX: now also TP71.1
- net BUTTON_N: now reaches U11.19 (GP14)
- net BUTTON_N: now also R83.2
- net GPS_TX: now reaches U11.2 (GP1)
- net GPS_TX: now also J71.4 (Pin_4)
- net VSYS: now reaches U11.39 (VSYS)
- net VSYS: now also JP41.3 (B)
- net VBUS: now reaches U11.40 (VBUS)
- net VBUS: now also JP41.1 (A)
- net SYNTH_SCL: now reaches U11.7 (GP5)
- net SYNTH_SCL: now also R32.2, U31.4 (SCL)
- net AMP_EN: now reaches U11.9 (GP6)
- net AMP_EN: now also R51.1, U51.3 (ON)
- net AMP_5V_IN: now reaches JP41.2 (C)
- net AMP_5V_IN: now also C41.1, C51.1, JP51.1 (A), U41.1 (IN), U41.3 (EN), U51.1 (VIN)
- net AMP_BIAS: now reaches RV61.2
- net AMP_BIAS: now also R62.1, C65.1
- net SYNTH_RF: now reaches C61.1
- net SYNTH_RF: now also U31.10 (CLK0)
- net RF_AC: now reaches C61.2
- net RF_AC: now also R61.1
- net AMP_DRAIN: now reaches C64.1
- net AMP_DRAIN: now also L61.2, Q61.1 (D)
- net TX_OUT: now reaches C64.2
- net TX_OUT: now also J61.1 (In)
- net AMP_GATE: now reaches R61.2
- net AMP_GATE: now also Q61.2 (G), R62.2, R63.1
- net GPS_PPS_RAW: now reaches R75.1
- net GPS_PPS_RAW: now also J71.3 (Pin_3)
- net AMP_CT: now reaches U51.4 (CT)
- net AMP_CT: now also C52.1
- net AMP_QOD: now reaches U51.5 (QOD)
- net AMP_QOD: now also R52.1
- no-connect marks 0 -> 20
Other:
- note added: "Always-on clock; independent AMP_EN."
- note added: "QLG3 underside male pins -> shield TOP female socket. 1=3V3 2=VBAT(3V3) 3=PPS 4=GPS_TX 5=GND"
- note removed: "Placement only: connections and PCB synchronization are pending. Always-on clock; independent AMP_EN. GP6 / GP14 / GP15 remain unapproved control candidates."
- note removed: "QLG3 header: 1 3V3 / 2 VBAT(3V3) / 3 PPS / 4 GPS_TX / 5 GND"
- moved on the sheet: C21, C22, C23, C31, C32, C41, C42, C51, C52, C53, C61, C62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

Commit message: Add single-post QLG3 variant and restore edge-launch SMA
Parts:
- J61: footprint wsprrypico-synth-shield:SMA_BAT_Wireless_BWSMA-KWE-Z001 -> wsprrypico-synth-shield:SMA_Adafruit_1865_EdgeMount; LCSC Part # C496551 -> (none); MPN BWSMA-KWE-Z001 -> 1865; Manufacturer BAT WIRELESS -> Adafruit; Selection status Selected prototype -> Existing project edge-mount footprint selected; manual fit; Specified Value 50 ohm SMA female; right angle -> 50 ohm SMA female; board-edge mount; 1.6 mm PCB; Supplier URL https://www.lcsc.com/product-detail/C496551.html -> https://www.adafruit.com/product/1865; Technology Coaxial connector -> Edge-launch coaxial connector
- J71: footprint wsprrypico-synth-shield:QLG3_GPS_UndersideHeader -> wsprrypico-synth-shield:QLG3_GPS_UndersideHeader_SinglePost
Changed lines of the file:
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@@
 			)
 		)
-		(property "Footprint" "wsprrypico-synth-shield:SMA_BAT_Wireless_BWSMA-KWE-Z001"
+		(property "Footprint" "wsprrypico-synth-shield:SMA_Adafruit_1865_EdgeMount"
 			(at 270.51 107.95 0)
 			(hide yes)
@@
 			)
 		)
-		(property "Datasheet" "https://www.lcsc.com/product-detail/C496551.html"
+		(property "Datasheet" "https://cdn-shop.adafruit.com/product-files/1865/C2387-001_datasheet.pdf"
 			(at 270.51 107.95 0)
 			(hide yes)
@@
 			)
 		)
-		(property "Description" "RF output after DC blocking; external LPF required; 50 ohm SMA female; right angle; Coaxial connector"
+		(property "Description" "RF output after DC blocking; external LPF required; Adafruit 1865 SMA female board-edge connector for 1.6 mm PCB"
 			(at 270.51 107.95 0)
 			(hide yes)
@@
 			)
 		)
-		(property "Manufacturer" "BAT WIRELESS"
+		(property "Manufacturer" "Adafruit"
 			(at 270.51 107.95 0)
 			(hide yes)
@@
 			)
 		)
-		(property "MPN" "BWSMA-KWE-Z001"
+		(property "MPN" "1865"
 			(at 270.51 107.95 0)
 			(hide yes)
@@
 			)
 		)
-		(property "LCSC Part #" "C496551"
+		(property "LCSC Part #" ""
 			(at 270.51 107.95 0)
 			(hide yes)
@@
 			)
 		)
-		(property "Supplier URL" "https://www.lcsc.com/product-detail/C496551.html"
+		(property "Supplier URL" "https://www.adafruit.com/product/1865"
 			(at 270.51 107.95 0)
 			(hide yes)
@@
 			)
 		)
-		(property "Specified Value" "50 ohm SMA female; right angle"
+		(property "Specified Value" "50 ohm SMA female; board-edge mount; 1.6 mm PCB"
 			(at 270.51 107.95 0)
 			(hide yes)
@@
 			)
 		)
-		(property "Technology" "Coaxial connector"
+		(property "Technology" "Edge-launch coaxial connector"
 			(at 270.51 107.95 0)
 			(hide yes)
@@
 			)
 		)
-		(property "Selection status" "Selected prototype"
+		(property "Selection status" "Existing project edge-mount footprint selected; manual fit"
 			(at 270.51 107.95 0)
 			(hide yes)
@@
 			)
 		)
-		(property "Footprint" "wsprrypico-synth-shield:QLG3_GPS_UndersideHeader"
+		(property "Footprint" "wsprrypico-synth-shield:QLG3_GPS_UndersideHeader_SinglePost"
 			(at 148.59 182.88 0)
 			(hide yes)
