File: WsprryPico Synth Shield with GPS/WsprryPico Synth Shield with GPS.kicad_pcb (KiCad board)
At the start: 2 copper layers, 53.3 x 22.9 mm, 46 parts, among them J61 SMA 50ohm, J71 U.FL 50ohm, Q61 BS170, SW11 Push, U21 TPS7A2033, U31 TPS22918, U51 Si5351A-B-GTR, U71 ATGM336H-5N31, Y41 25MHz TCXO

Commit message: Add silkscreen and version
Other:
- board text added: "WsprryPico Si5351 w/GPS Copyright © 2026 Lee C. Bussy [AA0NT] Version ${BOARD_REV}"
